File: smartmic/SM1000-C/SM1000-C.brd (EAGLE design)
At the start: 65 x 90 mm, 187 parts, among them CN1 HDR100-3, CN10 MJ-3523-SMT, CN11 HDR100-3, CN12 HRS-DF11-16DS, CN2 MOLEX-MINI-B-SMT, CN3 RASM722PX, CN4 RJ-45, CN5 MJ-3523-SMT, CN6 SJ-3524-SMT, CN7 MJ-3523-SMT, CN8 SJ-3524-SMT, CN9 MJ-3523-SMT, J1 JMP-2PIN, J3 JMP-2PIN, J4 JMP-2PIN, J5 JMP-2PIN, P1 TPAD50, P10 TPAD50, P11 TPAD50, P12 TPAD50, P13 TPAD50, P14 TPAD50, P15 TPAD50, P16 TPAD50, P17 TPAD50, P18 TPAD50, P19 TPAD50, P2 TPAD50, P20 TPAD50, P21 PAD070-035, P22 PAD070-035, P23 PAD070-035, P24 PAD070-035, P3 TPAD50, P4 TPAD50, P5 TPAD50, P6 TPAD50, P7 TPAD50, P8 TPAD50, P9 TPAD50, SW1 SW-BOURNS-7914S, SW2 SW-BOURNS-7914S, SW3 DPDT, SW4 SW-BOURNS-7914S, T1 SM-LP-5001, T2 SM-LP-5001, U1 STM32F405, U2 LD3985M33R, U3 STMPS2141, U4 EMIF02-USB03F2, U5 TPS54329E, U6 LMV341, U7 LMV341, U8 LM386M-1, U9 LMV341

Commit message: Update changes to SM1000-C schematic  RGB 09/26/14
Parts:
- removed J5: JMP-2PIN, _Coherix:JMPR-2PIN
- added R54, R55: 0 Ohm, AA-ipc-7351-resistor:RESC1608X55N
- added SW5: SW-BOURNS-7914J, SM1000:SW-BOURNS-7914J
- moved C57 155.0 mm to (68.0, 75.0)
Connections:
- new net N$29: R55.2, U1.29
- new net N$36: R54.2, U1.30
- net DAC1_OUT: now also R55.1; no longer U1.29
- net DAC2_OUT: now also R54.1; no longer U1.30
- net GND: now also SW5.1, SW5.2; no longer J5.1
- net NRST: now also SW5.3, SW5.4; no longer J5.2
Routing:
- net DAC1_OUT: track 34.0 -> 32.3 mm
- net DAC2_OUT: track 34.1 -> 32.6 mm

Commit message: Update file & add DIM PDFs  RGB 09/27/14
Parts:
- C57: value (none) -> 3.9nF,16V
- moved SW5 100.1 mm to (-14.5, 58.5)
- moved C28 35.9 mm to (-14.2, 50.2), turned to 180 degrees
- moved C29 35.4 mm to (-14.2, 53.2), turned to 180 degrees
- moved C24 34.0 mm to (-15.0, 69.8)
- moved C54 25.9 mm to (-14.0, 0.50)
- moved C13 25.4 mm to (-19.5, 19.6), turned to 0 degrees
- moved C12 22.8 mm to (-19.5, 22.3), turned to 0 degrees
- moved C25 20.6 mm to (-15.0, 46.5), turned to 0 degrees
- moved R10 20.5 mm to (-19.6, 25.1), turned to 180 degrees
- moved C11 18.3 mm to (-19.4, 28.2), turned to 0 degrees
- moved R18 17.6 mm to (-20.0, 43.0), turned to 0 degrees
- moved C10 17.5 mm to (-19.5, 31.2), turned to 0 degrees
- moved L1 17.4 mm to (-19.5, 34.0), turned to 180 degrees
- moved C57 17.0 mm to (79.5, 62.5)
- moved R21 14.7 mm to (-14.5, 42.0), turned to 0 degrees
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Other:
- board text added: "SM1000 Rev C"
- board text removed: "SM1000 Rev B1"

Commit message: Update changes to Schematic, etc. RGB 09/27/14
Parts:
- C25: value 22uF,25V,1210 -> 22uF,25V,3528,Tant; device ipc-7351-capacitor:CAPC3225X168N -> AA-ipc-7351-capacitor:CAPMP6032X280N
- C28, C29: value 10uF,25V,1206 -> 10uF,25V,3528,Tant; device ipc-7351-capacitor:CAPC3215X168N -> AA-ipc-7351-capacitor:CAPMP3528X210N
- R48: value 4.7K,1% -> 10K,1%
- SW1: device SM1000-2L-70x90:SW-BOURNS-7914S -> SM1000:SW-BOURNS-7914S
- moved C25 1.00 mm to (-14.0, 46.5)
Connections:
- net +5V: now also C28.+, C29.+; no longer C28.1, C29.1
- net +VIN: now also C25.+; no longer C25.1
- net GND: now also C25.-, C28.-, C29.-; no longer C25.2, C28.2, C29.2
Routing:
- net BOOT0: track 26.0 -> 22.0 mm
- net VDD: track 126.0 -> 122.0 mm

Commit message: Updates to schematic, PCB & Change-Log. RGB 10/02/14
Parts:
- removed C32: 2.2uF,16V, AA-ipc-7351-capacitor:CAPC1608X92N
- removed L1: FCM1608, _RoweTel:FCM1608
- removed L3: 100uH, _RoweTel:CBC3225T101MR
- removed P21, P22, P23, P24: PAD070-035, _Coherix:PAD070-035
- added D1: RSX051VA30, _RoweTel:TUMD2
- added FB5: (no value), _RoweTel:FE0805
- added R32: (no value), AA-ipc-7351-resistor:RESC1608X55N
- R39: value 2.21K,1% -> 4.7,0.5W,1206; device AA-ipc-7351-resistor:RESC1608X55N -> AA-ipc-7351-resistor:RESC3115X70N
- moved R39 33.5 mm to (82.5, 41.5), turned to 0 degrees
- moved C54 15.5 mm to (-14.5, 16.0)
- moved C55 15.5 mm to (-14.5, 33.5)
- moved C56 15.5 mm to (-14.5, 30.0)
- moved R29 15.5 mm to (-14.5, 20.0)
- moved R9 15.5 mm to (-14.5, 25.0)
- moved LD2 12.0 mm to (78.5, 34.5)
Connections:
- removed net APTT: C45.1, CN12.6, CN9.10
- removed net AVSS: C10.2, C11.2, C12.2, C13.2, C22.2, C23.2, C32.2, C34.2, C35.2, C41.2, C42.2, C50.2, C55.2, C56.2, C57.2, CN5.1, CN8.1, J4.2, MIC1.2, P23.1, R22.1, R40.2, R45.2, R46.1, R50.2, R52.1, T1.3, T2.3, U1.20, U6.2, U7.2, U8.2, U8.4, U9.2
- removed net MIC: C44.1, CN12.7, CN7.10
- removed net N$26: FB4.2, R11.1
- removed net N$33: FB1.1, T1.6
- removed net N$64: CN6.2, FB1.2
- removed net N$72: CN7.2, FB2.2
- removed net N$73: CN9.2, FB6.2
- removed net N$76: CN5.2, FB4.1
- removed net N$78: R48.2, T2.6
- removed net RF: C43.2, C44.2, C45.2, CN12.4, CN12.5, CN4.10, CN4.9, CN6.1, CN7.1, CN9.1, LD2.3, R49.1, T1.4, T2.4
- removed net SPKR: C43.1, CN12.8, CN6.4
- new net N$37: U8.6
- new net S$1: T1.3, T2.3
- new net S$2: R49.1
- net +5V: now also D1.C
- net +VIN: no longer U8.6
- net AVDD: no longer C32.1, P24.1
- net GND: now also C10.2, C11.2, C12.2, C13.2, C22.2, C23.2, C34.2, C35.2, C41.2, C42.2, C50.2, C55.2, C56.2, C57.2, J4.2, MIC1.2, R22.1, R40.2, R45.2, R46.1, R50.2, R52.1, U1.20, U6.2, U7.2, U8.2, U8.4, U9.2; no longer CN10.1, CN3.1, CN3.3, P22.1
- net N$24: no longer L3.2
- net N$25: no longer R39.1
- net N$30: now also D1.A
- net N$45: no longer R39.2
- net N$5: no longer L1.2
- net N$60: no longer CN5.10
- net N$62: no longer CN8.4
- net N$75: no longer CN8.2, CN8.3
- net N$77: no longer L3.1
- net N$79: now also C43.1
- net VDD: no longer L1.1, P21.1
Routing:
- net +VIN: track 84.2 -> 13.0 mm, vias 1 -> 0
- net AVSS: track 41.9 -> 0.00 mm, vias 6 -> 0
- net RF: track 47.7 -> 17.0 mm, vias 3 -> 0
- net GND: track 125.3 -> 146.7 mm, vias 34 -> 40
- net N$75: track 18.9 -> 0.00 mm
- net S$2: track 0.00 -> 11.5 mm
- net N$45: track 7.12 -> 0.00 mm
- net N$76: track 8.02 -> 4.00 mm
- net N$77: track 7.86 -> 11.5 mm
- net SPKR: track 3.32 -> 0.00 mm
- net N$8: track 51.3 -> 48.2 mm
- net MIC: track 2.82 -> 0.00 mm
- net APTT: track 33.8 -> 31.5 mm
- net N$26: track 2.23 -> 0.00 mm
- net N$39: track 29.3 -> 27.2 mm
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- removed copper zone on layer 1, net RF
- removed copper zone on layer 16, net RF

Commit message: Updateds per DRowe & Rbarnich  RGB 10/04/14 Schematic & PCB 10/04/14  10:56AM
Parts:
- moved CN10 47.2 mm to (8.00, 54.5), turned to 0 degrees
- moved SW1 1.50 mm to (2.50, 62.5), flipped to the bottom
Routing:
- net +VIN: track 13.0 -> 6.30 mm
- net N$70: track 15.6 -> 12.0 mm
Changed lines of the file:
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@@
 <layer number="14" name="Route14" color="1" fill="6" visible="no" active="no"/>
 <layer number="15" name="VDD" color="6" fill="1" visible="no" active="yes"/>
-<layer number="16" name="Bottom" color="1" fill="1" visible="no" active="yes"/>
+<layer number="16" name="Bottom" color="1" fill="1" visible="yes" active="yes"/>
 <layer number="17" name="Pads" color="2" fill="1" visible="yes" active="yes"/>
 <layer number="18" name="Vias" color="2" fill="1" visible="yes" active="yes"/>
@@
 <layer number="20" name="Dimension" color="15" fill="1" visible="yes" active="yes"/>
 <layer number="21" name="tPlace" color="7" fill="1" visible="yes" active="yes"/>
-<layer number="22" name="bPlace" color="7" fill="1" visible="no" active="yes"/>
+<layer number="22" name="bPlace" color="7" fill="1" visible="yes" active="yes"/>
 <layer number="23" name="tOrigins" color="15" fill="1" visible="yes" active="yes"/>
-<layer number="24" name="bOrigins" color="15" fill="1" visible="no" active="yes"/>
+<layer number="24" name="bOrigins" color="15" fill="1" visible="yes" active="yes"/>
 <layer number="25" name="tNames" color="7" fill="1" visible="yes" active="yes"/>
-<layer number="26" name="bNames" color="7" fill="1" visible="no" active="yes"/>
+<layer number="26" name="bNames" color="7" fill="1" visible="yes" active="yes"/>
 <layer number="27" name="tValues" color="7" fill="1" visible="no" active="yes"/>
 <layer number="28" name="bValues" color="7" fill="1" visible="no" active="yes"/>
@@
 <attribute name="VALUE" x="65.2875" y="64.775" size="1" layer="27" font="vector" ratio="10" rot="R90"/>
 </element>
-<element name="CN10" library="_RoweTel" package="MJ-3523-SMT" value="MJ-3523-SMT" x="16" y="8" smashed="yes" rot="MR270">
-<attribute name="NAME" x="12" y="8" size="1" layer="26" ratio="10" rot="MR270"/>
+<element name="CN10" library="_RoweTel" package="MJ-3523-SMT" value="MJ-3523-SMT" x="8" y="54.5" smashed="yes" rot="MR0">
+<attribute name="NAME" x="8" y="58.5" size="1" layer="26" ratio="10" rot="MR0"/>
 </element>
 <element name="R37" library="AA-ipc-7351-resistor" package="RESC1608X55N" value="2.2K,1%" x="44" y="66" locked="yes" smashed="yes" rot="R90">
@@
 <attribute name="NAME" x="10.83" y="71.64" size="0.8128" layer="25" ratio="10"/>
 </element>
-<element name="SW1" library="SM1000" package="SW-BOURNS-7914S" value="SW-BOURNS-7914S" x="2.5" y="61" smashed="yes" rot="R90">
-<attribute name="NAME" x="1.2" y="63.8" size="0.8128" layer="25" ratio="10"/>
+<element name="SW1" library="SM1000" package="SW-BOURNS-7914S" value="SW-BOURNS-7914S" x="2.5" y="62.5" smashed="yes" rot="MR90">
+<attribute name="NAME" x="3.8" y="65.3" size="0.8128" layer="26" ratio="10" rot="MR0"/>
 </element>
 <element name="R1" library="AA-ipc-7351-resistor" package="RESC1608X55N" value="10K,1%" x="15.5" y="62.5" locked="yes" smashed="yes">
@@
 <contactref element="R5" pad="1"/>
 <contactref element="R3" pad="1"/>
-<wire x1="1.34" y1="62.47" x2="3.66" y2="62.47" width="0.2" layer="1"/>
+<wire x1="3.66" y1="63.97" x2="1.34" y2="63.97" width="0.2" layer="16"/>
 <polygon width="0.2" layer="15" isolate="0.3">
 <vertex x="1" y="89"/>
@@
 <contactref element="R18" pad="2"/>
 <wire x1="22.2" y1="51.7" x2="24.13" y2="44.45" width="0" layer="19" extent="1-2"/>
-<wire x1="3.66" y1="62.47" x2="7.5" y2="62.5" width="0" layer="19" extent="1-1"/>
-<wire x1="-19.05" y1="43" x2="1.34" y2="62.47" width="0" layer="19" extent="1-1"/>
+<wire x1="1.34" y1="63.97" x2="7.5" y2="62.5" width="0" layer="19" extent="1-1"/>
+<wire x1="-19.05" y1="43" x2="3.66" y2="63.97" width="0" layer="19" extent="1-1"/>
 </signal>
 <signal name="BOOT1">
@@
 <wire x1="16" y1="61.5" x2="16.3" y2="61.8" width="0.2" layer="1"/>
 <wire x1="16.3" y1="61.8" x2="16.3" y2="62.5" width="0.2" layer="1"/>
-<wire x1="1.34" y1="59.53" x2="3.66" y2="59.53" width="0.2" layer="1"/>
-<wire x1="3.66" y1="59.53" x2="7" y2="61.5" width="0" layer="19" extent="1-1"/>
+<wire x1="3.66" y1="61.03" x2="1.34" y2="61.03" width="0.2" layer="16"/>
+<wire x1="1.34" y1="61.03" x2="7" y2="61.5" width="0" layer="19" extent="1-1"/>
 </signal>
 <signal name="N$1">
@@
 <wire x1="53.25" y1="79.75" x2="53.25" y2="80.2" width="0.2" layer="1"/>
 <contactref element="P20" pad="1"/>
-<wire x1="7" y1="59.07" x2="4.93" y2="57" width="0.4" layer="16"/>
-<wire x1="7.02" y1="59.07" x2="7" y2="59.07" width="0.4" layer="16"/>
-<wire x1="7.02" y1="59.07" x2="7.31" y2="59.36" width="0.4" layer="16"/>
-<wire x1="7.31" y1="59.36" x2="7.31" y2="59.86" width="0.4" layer="16"/>
-<wire x1="4.93" y1="57" x2="4.93" y2="54.16" width="0.4" layer="16"/>
 <contactref element="U5" pad="2"/>
 <contactref element="R34" pad="1"/>
@@
 <contactref element="C25" pad="+"/>
 <wire x1="7.31" y1="59.86" x2="50.135" y2="78.635" width="0" layer="19" extent="1-1"/>
-<wire x1="5.55" y1="43.4" x2="4.93" y2="54.16" width="0" layer="19" extent="1-16"/>
+<wire x1="5.55" y1="43.4" x2="7.31" y2="59.86" width="0" layer="19" extent="1-1"/>
+<wire x1="7.05" y1="41.05" x2="5.55" y2="43.4" width="0" layer="19" extent="1-1"/>
+<wire x1="11" y1="40" x2="7.05" y2="41.05" width="0" layer="19" extent="1-1"/>
+<wire x1="1.9" y1="41.1" x2="5.55" y2="43.4" width="0" layer="19" extent="1-1"/>
 <wire x1="-13.55" y1="42" x2="1.9" y2="41.1" width="0" layer="19" extent="1-1"/>
 <wire x1="-16.45" y1="46.5" x2="-13.55" y2="42" width="0" layer="19" extent="1-1"/>
@@
 <wire x1="47" y1="60" x2="47" y2="59.5" width="0.2" layer="1"/>
 <wire x1="47" y1="59.5" x2="48" y2="58.5" width="0.2" layer="1"/>
-<wire x1="12.4" y1="11.8" x2="54.15" y2="29.05" width="0" layer="19" extent="1-16"/>
+<wire x1="11.8" y1="58.1" x2="54.15" y2="29.05" width="0" layer="19" extent="1-16"/>
 </signal>
 <signal name="N$70">
@@
 <wire x1="5.5" y1="64.5" x2="4.75" y2="65.25" width="1.27" layer="16"/>
 <wire x1="4.75" y1="65.25" x2="4.75" y2="68.5" width="1.27" layer="16"/>
-<wire x1="5.5" y1="59.27" x2="3" y2="56.77" width="1.27" layer="16"/>
+<wire x1="5.5" y1="59.27" x2="3" y2="56.77" width="0" layer="19" extent="1-16"/>
 <contactref element="R21" pad="1"/>
 <wire x1="-15.45" y1="42" x2="3" y2="56.77" width="0" layer="19" extent="1-16"/>
