File: smartmic/SM1000-D/RELEASE/SM1000-D.sch (EAGLE design)
At the start: 196 parts, among them CN1 HDR100-3, CN10 ST-3509, CN11 HDR100-3, CN12 HRS-A3C-16DA, CN2 JS-MU3-002, CN3 DS-0518, CN4 RJ-45, CN5 ST-3509, CN6 ST-3509, CN7 ST-3509, CN8 ST-3509, CN9 ST-3509, J1 JMP-2PIN, J3 JMP-2PIN, J4 JMP-2PIN, P1 TPAD50, P10 TPAD50, P11 TPAD50, P12 TPAD50, P13 TPAD50, P14 TPAD50, P16 TPAD50, P18 TPAD50, P19 TPAD50, P2 TPAD50, P20 TPAD50, P3 TPAD50, P4 TPAD50, P5 TPAD50, P6 TPAD50, P7 TPAD50, P8 TPAD50, P9 TPAD50, SW1 SW-SPDT-8US8WR2C2M7RES, SW2 TS-026, SW3 DPDT, SW4 TS-026, SW5 TS-02B, T1 SM-LP-5001, T2 SM-LP-5001, U1 STM32F405VGT6, U2 LD3985M33R, U3 STMPS2141, U4 EMIF02-USB03F2, U5 TPS54329E, U6 LMV341, U7 LMV341, U8 LM386M-1, U9 LMV341

Commit message: Production Release of SM1000-D PCB files
Parts:
- PCB1: value SM1000C -> SM1000D
- R42: value 500K,POT -> 500K,TrimPOT
- R47: value 500,POT -> 500,TrimPOT
- R52: value 1K,POT -> 1K,TrimPOT
Other:
- note added: "01-23-15"
- note added: "01/23/15"
- note added: "MISC. PARTS"
- note added: "RELEASE REV. D TO PRODUCTION"
- note added: "RELEASE REV. D TO PRODUCTION."
- note removed: "04/21/14"
- note removed: "04/25/14"
- note removed: "05/28/14"
- note removed: "06/13/14"
- note removed: "11/18/14"
- note removed: "A"
- note removed: "Added to SourceForge Repository"
- note removed: "B"
- note removed: "C"
- note removed: "Pre-Release to Prototype"
- note removed: "Release for Production"
- note removed: "Release for Prototype"
- note removed: "Release for Review"
- moved on the sheet: PCB1
