File: sm2000/CAD/SM2000.sch (EAGLE design)
At the start: 361 parts, among them CN1 HDR100-3, CN10 ST-3509, CN11 HDR100-3, CN2 JS-MU3-002, CN3 DS-0518, CN5 ST-3509, CN8 ST-3509, J1 JMP-2PIN, J2 JMP-2PIN, J3 JMP-2PIN, J4 CONN-BOOM-XH-2A, P10 TPAD50, P11 TPAD50, P12 TPAD50, P13 TPAD50, P14 TPAD50, P16 TPAD50, P18 TPAD50, P19 TPAD50, P20 TPAD50, P21 TPAD50, P3 TPAD50, P4 TPAD50, P5 TPAD50, P6 TPAD50, P7 TPAD50, P8 TPAD50, P9 TPAD50, Q1 MMBT3904, Q10 MMBT3904, Q11 STR2P3LLH6, Q12 BRF92, Q13 BFQ19, Q14 RD01MUS2, Q15 MMBT3904, Q17 MMT2904, Q18 MMT2904, Q2 MMBT3904, Q3 MMBT3904, Q4 MMBT3904, Q5 MMBT3904, Q6 MMBT3904, Q7 BC548, Q8 BC549, Q9 STR2P3LLH6, SW1 SW-LC2259, SW2 TS-026, SW3 SW-LC2259EENP, SW4 TS-026, SW5 TS-02B, U1 STM32F405VGT6, U10 DNL, U11 L78MXX, U12 PGA-103+, U13 ADE-1, U14 SI570CAC000141DG, U15 SI5351A, U2 L78MXX, U3 STMPS2141, U4 EMIF02-USB03F2, U5 L78MXX, U6 LD3985M33R, U7 SA612A, U8 LM386M-1, U9 LMV341, X1 BU-SMA-H, X2 BU-SMA-H

Commit message: 
Parts:
- C42, C43, C44: value 0.1u -> 0.1uF,25V
- C67, C68, C69, C71, C72, C73, C74, C75, C76: value 100nF -> 100nF,25V
- L20: value 5.7uH +/- 10% Q>20 -> 5.7uH
- L21: value 9.2uH +/- 10% Q>20 -> 9.2uH
- L22: value 5.2uH +/- 10% Q>20 -> 5.2uH
- L23: value 15uH +/- 10% Q>20 -> 15uH
- Q17, Q18: value MMT2904 -> MMBT3904
- U14: value SI570CAC000141DG -> SI570
- XTAL5: value 25MHz 10pF e.g. TXC 7B-25.000MEEQ-T -> 25MHz,TXC,SMD
Connections:
- removed net 3V3: FB13.1, FB22.1
- removed net N$117: FB16.1
- new net N$56: L20.1
- new net SCL: U14.SCL, U15.SCL
- new net SDA: U14.SDA, U15.SDA
- net +12V_RX: no longer Q11.D
- net +3.3V: now also FB13.1, FB16.1, FB22.1
- net N$40: now also Q11.D
Other:
- note added: "5.2uH +/- 10% Q>20"
- note added: "L20 5.7uH +/- 10% Q>20"
- note added: "L21 9.2uH +/- 10% Q>20"
- note added: "L23 15uH +/- 10% Q>20"
- note added: "Note: Have to hook up I2C lines on Si570 & Si5351A"
- note added: "Note: L22"
- note removed: "Rick: I cant find part designator/value?"
- note removed: "TX 2ND LO"
- moved on the sheet: C120, C121, C122, C125, C126, C132, C43, C44, FB13, FB15, FB16, FB22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
