File: sm2000/CAD/SM2000.sch (EAGLE design)
At the start: 382 parts, among them CN1 HDR100-3, CN10 ST-3509, CN11 HDR100-3, CN2 JS-MU3-002, CN3 DS-0518, CN5 ST-3509, CN8 ST-3509, J1 JMP-2PIN, J10 JMPR-2X2, J11 JMPR-2X2, J12 JMPR-2X2, J13 JMPR-2X2, J2 JMP-2PIN, J3 JMP-2PIN, J4 CONN-BOOM-XH-2A, J5 JMPR-2X2, J6 JMPR-2X2, J7 JMPR-2X2, J8 JMPR-2X2, J9 JMPR-2X2, P10 TPAD50, P11 TPAD50, P12 TPAD50, P13 TPAD50, P14 TPAD50, P16 TPAD50, P18 TPAD50, P19 TPAD50, P20 TPAD50, P21 TPAD50, P3 TPAD50, P4 TPAD50, P5 TPAD50, P6 TPAD50, P7 TPAD50, P8 TPAD50, P9 TPAD50, Q1 MMBT3904, Q10 MMBT3904, Q11 STR2P3LLH6, Q12 BRF92, Q13 BFQ19, Q14 RD01MUS2, Q15 MMBT3904, Q17 MMBT3904, Q18 MMBT3904, Q2 MMBT3904, Q3 MMBT3904, Q4 MMBT3904, Q5 MMBT3904, Q6 MMBT3904, Q7 MMBT3904, Q8 MMBT3906, Q9 STR2P3LLH6, SW1 SW-LC2259, SW2 TS-026, SW3 SW-LC2259EENP, SW4 TS-026, SW5 TS-02B, U1 STM32F405VGT6, U10 DNL, U11 L78MXX, U12 PGA-103+, U13 ADE-1, U14 SI570, U15 SI5351A, U17 TPS54329E, U2 L78MXX, U3 STMPS2141, U4 EMIF02-USB03F2, U6 LD3985M33R, U7 SA612A, U8 LM386M-1, U9 LMV341

Commit message: Changes to schematics per emails of 1/12/2016 - 1/14/2016 per David Rowe.
Parts:
- removed C101: 10nF,25V, _RoweTel:CAP-0805
- removed P5, P6, P7, P8: TPAD50, _Coherix:TPAD50
- added C38: 100uF,25V,EL, _RoweTel:CAP-CHEMI-F80
- added C41: 0.1uF.25V, _RoweTel:CAP-0805
- added J14: HDR100-5, _RoweTel:HDR100-5
- added L2: RFC, _RoweTel:RFC
- added LED10, LED11, LED5, LED6, LED7: SML-LX0603GW, _RoweTel:SML-LX0603SRW
- added LED8: SML-LX0603SRW, _RoweTel:SML-LX0603SRW
- added LED9: SML-LX0603YW, _RoweTel:SML-LX0603SRW
- added R100, R52: 1K,1%, _RoweTel:RES-0805
- added R116: 680,1%, _RoweTel:RES-0805
- added R117, R44, R51: 320,1%, _RoweTel:RES-0805
- added R23, R43, R9: 10K,1%, _RoweTel:RES-0805
- added R36: 1.5K,1%, _RoweTel:RES-0805
- added U5: LMV341, _RoweTel:LMV341
- added X1: BU-SMA-H, _RoweTel:BU-SMA-H
- C1: value 100nF,25V -> 22uF,25V; device _RoweTel:CAP-0805 -> _RoweTel:CAP-1210
- C103: value 100nF,25V -> 1nF,25V
- C136: value 1uF,25V -> 1uF,25V,EL
- C29: value CAP-10UF-WJ5 -> 1nF,25V; device _RoweTel:CAP-10UF-WJ5 -> _RoweTel:CAP-0805
- C5: value CAP-10UF-WJ5 -> 0.1uF.25V; device _RoweTel:CAP-10UF-WJ5 -> _RoweTel:CAP-0805
- C94: device rcl:C-EU025-024X044 -> _RoweTel:CAP-0805
- L10, L12, L14, L15, L16, L17, L18, L19, L25, L26, L9: device rcl:L-US0204/5 -> _RoweTel:L-ROWE_15X10
- L11, L13: device inductor-neosid:Z14/40CCW -> _RoweTel:RFC
- L20, L21, L22, L23: device rcl:L-US0204/5 -> _RoweTel:L-TDK-MLF-2012
- Q12: device transistor:-NPN-SOT23-EBC -> _RoweTel:BFR92
- Q13: device transistor:-NPN-SOT23-EBC -> _RoweTel:BFQ19
- R18, R34: value 10K,1/8W,5% -> 10K,1%
- R61, R62: value DNL -> 4.7K,1%
- U6: value LD3985M33R -> AP7215Y-33; device _RoweTel:LD3985 -> _RoweTel:AP7215Y
Connections:
- net TXDAC renamed TX_DAC
- removed net +12V: FB10.2, FB14.2, FB15.1
- removed net +12V_RX: R45.1
- removed net +3.3V: C8.1, FB13.1, FB16.1, FB22.1, U11.OUT
- removed net AVDD: C22.1, C35.1, C5.1, C6.1, C65.1, FB7.1, J3.2, R38.2, U6.VOUT, U9.!SHDN!, U9.V+
- removed net SCL: U14.SCL, U15.SCL
- removed net SDA: U14.SDA, U15.SDA
- removed net VDD: C16.1, C17.1, C18.1, C19.1, C20.1, C21.1, C52.1, C53.1, P13.1, R2.1, R24.1, R25.2, R3.1, R31.1, R37.1, R4.1, R5.1, R61.1, R62.1, R7.2, R8.2, SW1.2, SW1.5, U10.VCC, U1B.VDD1, U1B.VDD12, U1B.VDD2, U1B.VDD3, U1B.VDD4, U1B.VDD5
- new net +12VTXENB: R18.1
- new net 3V3: C16.1, C17.1, C18.1, C19.1, C20.1, C21.1, C52.1, C53.1, C8.1, FB13.1, FB16.1, FB22.1, P13.1, R2.1, R24.1, R25.2, R3.1, R31.1, R37.1, R4.1, R44.2, R5.1, R61.1, R62.1, R7.2, R8.2, SW1.2, SW1.5, U10.VCC, U11.OUT, U1B.VDD1, U1B.VDD12, U1B.VDD2, U1B.VDD3, U1B.VDD4, U1B.VDD5
- new net A3V3: C22.1, C35.1, C6.1, C65.1, FB21.2, FB7.1, J3.2, R38.2, R51.2, U5.!SHDN!, U5.V+, U6.OUT, U9.!SHDN!, U9.V+
- new net N$128: R43.1, R9.1, U5.-IN
- new net N$129: J8.1
- new net N$130: C29.1, C5.1, L11.1, L2.1
- new net N$131: LED8.A, R52.1
- new net N$132: LED6.A, R44.1
- new net N$134: LED10.A, R116.1
- new net N$138: LED11.A, R117.1
- new net N$63: LED5.A, R36.1
- new net VGG_DAC: U5.+IN
- net +12VRXENB: no longer R18.1
- net +5V: now also FB10.2, FB14.2, FB15.1, R116.2
- net +9V: now also C38.1, C41.1, L2.2, R36.2; no longer L11.2
- net +VIN: now also R117.2
- net ANT_SMA: now also X1.1; no longer J9.2
- net GND: now also C38.2, C41.2, J14.1, LED10.C, LED11.C, LED5.C, LED6.C, LED7.C, LED8.C, LED9.C, R23.1, R43.2, U5.GND; no longer C101.2
- net N$127: now also LED7.A, R51.1; no longer C101.1, U6.BYBASS
- net N$133: now also LED9.A, R100.1; no longer FB21.2
- net N$158: now also R23.2
- net N$19: now also L13.2; no longer L13.1
- net N$32: now also L11.2; no longer L11.1
- net N$54: now also U6.IN; no longer C29.1, U6.INH, U6.VIN
- net PA_OUTPUT: now also J9.2
- net PE0: now also J14.2; no longer P5.1
- net PE1: now also J14.3; no longer P6.1
- net PE2: now also J14.4; no longer P7.1
- net PE3: now also J14.5; no longer P8.1
- net RX+12V: now also R45.1, R52.2
- net SCL3: now also U14.SCL, U15.SCL
- net SDA3: now also U14.SDA, U15.SDA
- net TIAOUT: now also L20.1
- net TIA_OUT: no longer L20.1
- net TX+12V: now also L13.1, R100.2; no longer L13.2
- net VGG: now also R9.2, U5.OUT
Other:
- note added: "+5V -> 3V3"
- note added: "+5V -> A3V3"
- note added: "Need to adjust components in +5V reg for higher current."
- note added: "Vin -> 5.0VDC"
- note removed: "12 - 15VDC -> 5.0VDC"
- note removed: "12V for TX"
- note removed: "4.7K,1%"
- note removed: "5.0V -> 3.3V PS"
- note removed: "ARE Q17 & Q18 MMT2905s ?"
- note removed: "VDD -> AVDD"
- moved on the sheet: C1, C103, C107, C108, C109, C110, C111, C112, C113, C114, C115, C116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

Commit message: Cleaned up schematic. Ran ERC with no errors. Started arranging parts on board. Have to add scope test points. A lot of parts to fit on PCB! RGB
Parts:
- removed C137, C147, C148, C149: 1nF,25V, _RoweTel:CAP-0805
- removed C138: 12pF,50V, _RoweTel:CAP-0805
- removed C139, C140: 3.3pF,50V, _RoweTel:CAP-0805
- removed C144: 2.2pF,50V, _RoweTel:CAP-0805
- removed C145: 22pF,50V, _RoweTel:CAP-0805
- removed C146: 22pF,25V, _RoweTel:CAP-0805
- removed C150, C179: 22uF,25V, _RoweTel:CAP-1210
- removed C164: 100nF,25V, _RoweTel:CAP-0805
- removed C167: 22uF,25V,1210, AA-ipc-7351-capacitor:CAPACITOR_1210
- removed CN10: ST-3509, _RoweTel:ST-3509
- removed CN11: HDR100-3, _Coherix:HDR100-3
- removed D11, D12: BAR64-02V, _RoweTel:BAR64-02V
- removed FB20, FB21, FB22: FB0805, _RoweTel:FB0805
- removed L21: 9.2uH, _RoweTel:L-TDK-MLF-2012
- removed L22: 5.2uH, _RoweTel:L-TDK-MLF-2012
- removed L23: 15uH, _RoweTel:L-TDK-MLF-2012
- removed L25: 53nH 3T 5mm ID, _RoweTel:L-ROWE_15X10
- removed L26: 220nH, _RoweTel:L-ROWE_15X10
- removed P16, P18, P20, P21: TPAD50, _Coherix:TPAD50
- removed Q18: MMBT3904, transistor:-NPN-SOT23-EBC
- removed R127: 124.0K,1%, AA-ipc-7351-resistor:RESISTOR_0402
- removed R128: 22.1K,1%, AA-ipc-7351-resistor:RESISTOR_0402
- removed R129: 10K,1%, AA-ipc-7351-resistor:RESISTOR_0402
- removed SH4, SH5: SHUNT, _RoweTel:SHUNT
- removed U17: TPS54329E, _RoweTel:TPS54329E
- removed XTAL5: 25MHz,TXC,SMD, _RoweTel:XTAL-FY0800035
- added C101: 1pF,50V, _RoweTel:CAP-0805
- added C102, C106: 1nF,25V, _RoweTel:CAP-0805
- added C104, C84: 0.1uF.25V, _RoweTel:CAP-0805
- added C105: 33pF,50V, _RoweTel:CAP-0805
- added C45, C61, C70: 100nF,25V, _RoweTel:CAP-0805
- added C47: 8.2nF,25V, ipc-7351-capacitor:CAPACITOR_0603
- added C48: 100nF,25V, AA-ipc-7351-capacitor:CAPACITOR_0402
- added C50: 3.9nF,16V, _RoweTel:CAP-0805
- added C64: 12pF.50V, _RoweTel:CAP-0805
- added C66: 0.5pF,50V, _RoweTel:CAP-0805
- added CN4: JS-MU3-002, _RoweTel:JS-MU3-002
- added CN6: ST-3509, _RoweTel:ST-3509
- added D5: DNL, _RoweTel:PTVS20VP1UP
- added D6: BAR64-02V, _RoweTel:BAR64-02V
- added FB1, FB12, FB2: FB0805, _RoweTel:FB0805
- added L3, L5, L8: 68nH, _RoweTel:L-ROWE_15X10
- added L4: 57nH, _RoweTel:L-ROWE_15X10
- added L6: 168nH, _RoweTel:L-ROWE_15X10
- added P1, P6, P7, P8: TPAD50, _Coherix:TPAD50
- added Q16: MMBT3904, _RoweTel:MMBT3904
- added R118: 3.3K,1%, _RoweTel:RES-0805
- added R119: 100,1%, _RoweTel:RES-0805
- added R120: 10,1%, _RoweTel:RES-0805
- added U16: SA612A, _RoweTel:SA612A
- added XTAL4: ECS-10.7-15B, _RoweTel:ECS-10.7-15B
- C1: value 22uF,25V -> 100nF,25V; device _RoweTel:CAP-1210 -> _RoweTel:CAP-0805
- C10: value 1uF,16V -> 1nF,25V
- C100: value 33pF,50V -> 1nF,25V
- C107: value 100nF,25V -> 47pF,50V; device AA-ipc-7351-capacitor:CAPACITOR_0402 -> _RoweTel:CAP-0805
- C108: value 20pF,50V -> 0.1uF.25V; device AA-ipc-7351-capacitor:CAPACITOR_0402 -> _RoweTel:CAP-0805
- C109: value 8.2nF,25V -> 100uF,25V,EL; device ipc-7351-capacitor:CAPACITOR_0603 -> _RoweTel:CAP-CHEMI-F80
- C110: value 12pF.50V -> 33pF,50V
- C111: value 3.3pF,50V -> 0.1uF,25V
- C112: value 3.3pF,50V -> 39pF,50V
- C113: value 12pF,50V -> 0.1uF,25V
- C114: value 0.5pF,50V -> 0.1uF,25V
- C115: value 1nF,25V -> 5.6pF,50V
- C116: value 1nF,25V -> 2-12pF; device _RoweTel:CAP-0805 -> c-trimm:C-TRIMM3008
- C117, C133, C134: value 1nF,25V -> 0.1uF,25V
- C119: value 10uF,25V,EL -> 0.1uF,25V; device _RoweTel:CAP-10UF-WJ5 -> _RoweTel:CAP-0805
- C12, C24: value 1uF,16V -> 100nF,25V
- C120: value 39pF,50V -> 0.1uF,25V
- C122: value 5.6pF,50V -> 10uF,25V,EL; device _RoweTel:CAP-0805 -> _RoweTel:CAP-10UF-WJ5
- C123: value 2-12pF -> 27pF,50V; device c-trimm:C-TRIMM3008 -> _RoweTel:CAP-0805
- C124: value 0.1uF,25V -> 150pF,50V
- C125: value 0.1uF,25V -> 0.1uF.25V
- C126: value 0.1uF,25V -> 10uF,25V,EL; device _RoweTel:CAP-0805 -> _RoweTel:CAP-10UF-WJ5
- C127: value 27pF,50V -> 0.1uF,25V
- C129: value 0.1uF.25V -> 10uF,25V,EL; device _RoweTel:CAP-0805 -> _RoweTel:CAP-10UF-WJ5
- C13, C72, C73, C74, C75, C76: value 100nF,25V -> 1nF,25V
- C130: value 1nF,25V -> 10uF,25V,EL; device _RoweTel:CAP-0805 -> _RoweTel:CAP-10UF-WJ5
- C131, C78: value 0.1uF,25V -> 1nF,25V
- C132: value 150pF,50V -> 1nF,25V
- C136: value 1uF,25V,EL -> 10uF,25V,EL; device _RoweTel:CAP-TANT-1206 -> _RoweTel:CAP-10UF-WJ5
- C14, C35: value 2.2uF,16V -> 100nF,25V
- C15: value 2.2uF,16V -> 10nF,25V
- C16, C6: value 100nF,25V -> 1uF,16V
- C17: value 10nF,25V -> 2.2uF,16V
- C18: value 100nF,25V -> 2.2uF,16V
- C19, C21: value 10nF,25V -> 20pF,50V
- C2: value 20pF,50V -> 10nF,25V
- C22: value 100nF,25V -> 4.7uF,16V,TANT; device _RoweTel:CAP-0805 -> _RoweTel:CAP-TANT-1206
- C23: value 100nF,25V -> CAP-10UF-WJ5; device _RoweTel:CAP-0805 -> _RoweTel:CAP-10UF-WJ5
- C25: value 1pF,50V -> 10nF,25V
- C26: value 1nF,25V -> CAP-10UF-WJ5; device _RoweTel:CAP-0805 -> _RoweTel:CAP-10UF-WJ5
- C27: value 1nF,25V -> 1nF,25V,0402
- C28: value 100nF,25V -> 220nF,25V
- C29, C56: value 1nF,25V -> 100nF,25V
- C3: value 20pF,50V -> 100nF,25V
- C30: value 10nF,25V -> 100nF,25V
- C31: value CAP-10UF-WJ5 -> 100uF,6.3V,EL; device _RoweTel:CAP-10UF-WJ5 -> _RoweTel:NICHICON-WX-6.3
- C33: value 220nF,25V -> 100nF,25V
- C34: value 1nF,25V,0402 -> 220uF,25V; device _RoweTel:CAP-0805 -> _RoweTel:CAP-CHEMI-MVE-HA0
- C36: value 1nF,25V -> 22uF,25V; device _RoweTel:CAP-0805 -> _RoweTel:CAP-1210
- C37: value 100nF,25V -> 1nF,25V; device AA-ipc-7351-capacitor:CAPACITOR_0402 -> _RoweTel:CAP-0805
- C38: value 100uF,25V,EL -> 2.2uF,16V; device _RoweTel:CAP-CHEMI-F80 -> _RoweTel:CAP-0805
- C39: value 220uF,25V -> 100pF,50V; device _RoweTel:CAP-CHEMI-MVE-HA0 -> _RoweTel:CAP-0805
- C40: value 47nF,25V -> 1nF,25V
- C41: value 0.1uF.25V -> 100nF,25V
- C42, C43: value 0.1uF,25V -> 22uF,25V; device _RoweTel:CAP-0805 -> _RoweTel:CAP-1210
- C44: value 0.1uF,25V -> 1uF,25V
- C49: device _RoweTel:CAP-0805 -> AA-ipc-7351-capacitor:CAPACITOR_0402
- C5: value 0.1uF.25V -> 10nF,25V
- C51: value 100nF,25V -> 20pF,50V; device _RoweTel:CAP-0805 -> AA-ipc-7351-capacitor:CAPACITOR_0402
- C52: value 100nF,25V -> 220uF,25V; device _RoweTel:CAP-0805 -> _RoweTel:CAP-CHEMI-MVE-HA0
- C53: value 10nF,25V -> 47nF,25V
- C54: value 100pF,50V -> 22uF,25V,1210; device _RoweTel:CAP-0805 -> AA-ipc-7351-capacitor:CAPACITOR_1210
- C55: value 1nF,25V -> 220uF,25V; device _RoweTel:CAP-0805 -> _RoweTel:CAP-CHEMI-MVE-HA0
- C57: value 3.9nF,16V -> 100nF,25V
- C59: value 100uF,6.3V,EL -> 100nF,25V; device _RoweTel:NICHICON-WX-6.3 -> _RoweTel:CAP-0805
- C60, C63: value 220uF,25V -> 100nF,25V; device _RoweTel:CAP-CHEMI-MVE-HA0 -> _RoweTel:CAP-0805
- C62, C69: value 100nF,25V -> 3.3pF,50V
- C65: value 1uF,25V -> 100nF,25V
- C67: value 100nF,25V -> 12pF,50V
- C7: value CAP-10UF-WJ5 -> 1uF,16V; device _RoweTel:CAP-10UF-WJ5 -> _RoweTel:CAP-0805
- C77: value 0.1uF,25V -> 1uF,25V,EL; device _RoweTel:CAP-0805 -> _RoweTel:CAP-TANT-1206
- C79: value 10uF,25V,EL -> 22pF,50V; device _RoweTel:CAP-10UF-WJ5 -> _RoweTel:CAP-0805
- C80: value 10uF,25V,EL -> 3.3pF,50V; device _RoweTel:CAP-10UF-WJ5 -> _RoweTel:CAP-0805
- C81: value 10uF,25V,EL -> 1nF,25V; device _RoweTel:CAP-10UF-WJ5 -> _RoweTel:CAP-0805
- C82: value 10uF,25V,EL -> 12pF,50V; device _RoweTel:CAP-10UF-WJ5 -> _RoweTel:CAP-0805
- C87: value 22pF,50V -> 5.6pF,50V
- C88: value 1nF,25V -> 2.2pF,50V
- C89: value 5.6pF,50V -> 3.3pF,50V
- C9: value 4.7uF,16V,TANT -> 10nF,25V; device _RoweTel:CAP-TANT-1206 -> _RoweTel:CAP-0805
- C90: value 1nF,25V -> 0.1uF.25V
- C91, C97: value 0.1uF.25V -> 1nF,25V
- C92: value 0.1uF.25V -> 22pF,50V
- C93: value 33pF,50V -> 22pF,50V
- C94: value 22pF,50V -> 0.1uF.25V
- C95: value 1nF,25V -> 22pF,25V
- C99: value 47pF,50V -> 1nF,25V
- CN2: value JS-MU3-002 -> ST-3509; device _RoweTel:JS-MU3-002 -> _RoweTel:ST-3509
- CN3: value DS-0518 -> HDR100-3; device _RoweTel:DS-0518 -> _Coherix:HDR100-3
- CN5: value ST-3509 -> DS-0518; device _RoweTel:ST-3509 -> _RoweTel:DS-0518
- D1: value PTVS20VP1UP -> DNL; device _RoweTel:PTVS20VP1UP -> _RoweTel:PESD5ZX
- D10: value BAR64-02V -> BAT18; device _RoweTel:BAR64-02V -> _RoweTel:BAT18
- D2: value BAT60J -> DNL; device _RoweTel:BAT60J -> _RoweTel:PESD5ZX
- D3: value DNL -> PTVS20VP1UP
- D4: value BAT18 -> BAT60J; device _RoweTel:BAT18 -> _RoweTel:BAT60J
- D7, D8: value DNL -> BAR64-02V; device _RoweTel:PESD5ZX -> _RoweTel:BAR64-02V
- J14: value HDR100-5 -> JMPR-2X2; device _RoweTel:HDR100-5 -> _RoweTel:JMPR-2X2
- J2: value JMP-2PIN -> HDR100-5; device _Coherix:JMP-2PIN -> _RoweTel:HDR100-5
- J5: value JMPR-2X2 -> JMP-2PIN; device _RoweTel:JMPR-2X2 -> _Coherix:JMP-2PIN
- L10: value 168nH -> 53nH 3T 5mm ID
- L11: value RFC -> 220nH; device _RoweTel:RFC -> _RoweTel:L-ROWE_15X10
- L12: value 54nH -> RFC; device _RoweTel:L-ROWE_15X10 -> _RoweTel:RFC
- L15: value 57nH -> RFC; device _RoweTel:L-ROWE_15X10 -> _RoweTel:RFC
- L16: value 68nH -> 57nH
- L17: value 68nH -> 5.7uH; device _RoweTel:L-ROWE_15X10 -> _RoweTel:L-TDK-MLF-2012
- L18: value 68nH -> 9.2uH; device _RoweTel:L-ROWE_15X10 -> _RoweTel:L-TDK-MLF-2012
- L19: value 68nH -> 5.2uH; device _RoweTel:L-ROWE_15X10 -> _RoweTel:L-TDK-MLF-2012
- L2: value RFC -> 68nH; device _RoweTel:RFC -> _RoweTel:L-ROWE_15X10
- L20: value 5.7uH -> 15uH
- L9: value 57nH -> 54nH
- LED11: value SML-LX0603GW -> SML-LX0603YW
- LED8: value SML-LX0603SRW -> SML-LX0603GW
- LED9: value SML-LX0603YW -> SML-LX0603SRW
- Q11: value STR2P3LLH6 -> BRF92; device _RoweTel:STR2P3LLH6 -> _RoweTel:BFR92
- Q12: value BRF92 -> BFQ19; device _RoweTel:BFR92 -> _RoweTel:BFQ19
- Q13: value BFQ19 -> RD01MUS2; device _RoweTel:BFQ19 -> _RoweTel:RD01MUS2
- Q14: value RD01MUS2 -> MMBT3904; device _RoweTel:RD01MUS2 -> transistor:-NPN-SOT23-EBC
- Q15: device _RoweTel:MMBT3904 -> transistor:-NPN-SOT23-EBC
- Q17: value MMBT3904 -> MMBT3906; device transistor:-NPN-SOT23-EBC -> transistor-pnp:2N2905
- Q2, Q4: value MMBT3904 -> STR2P3LLH6; device _RoweTel:MMBT3904 -> _RoweTel:STR2P3LLH6
- Q8: value MMBT3906 -> MMBT3904; device transistor-pnp:2N2905 -> _RoweTel:MMBT3904
- Q9: value STR2P3LLH6 -> MMBT3904; device _RoweTel:STR2P3LLH6 -> _RoweTel:MMBT3904
- R1, R55, R74: value 10K,1% -> 680,1%
- R10: value 47,1% -> 4.7K,1%
- R102, R84: value 1K,1% -> 150,1%
- R103: value 1K,1% -> 33K,1%
- R104: value 150,1% -> 15K,1%
- R105: value 0 Ohm -> 3K,1%
- R106, R107: value 0 Ohm -> 1K,1%
- R108: value 3K,1% -> 10,1%
- R109: value 1K,1% -> 49.9,1%
- R11: value 100,1% -> 1K,1%; device AA-ipc-7351-resistor:RESISTOR_0603 -> _RoweTel:RES-0805
- R110: value 10,1% -> 39K,1%
- R111: value 33K,1% -> 18K,1%
- R112: value 15K,1% -> 2.2K,1%
- R114: value 49.9,1% -> 100,1%
- R115: value 150,1% -> 10,1%
- R116: value 680,1% -> 150,1%
- R117: value 320,1% -> 3.3K,1%
- R12: value 680,1% -> 47,1%
- R13, R16: value 680,1% -> 0 Ohm
- R14: value 220,1% -> 0 Ohm
- R15: value 680,1% -> 220,1%
- R17: value 2.2K,1/8W,5% -> 10K,1%
- R19: value 22,1% -> 470,1%; device _RoweTel:RES-0805 -> AA-ipc-7351-resistor:RESISTOR_0402
- R2, R3, R4: value 4.7K,1% -> 680,1%
- R20: value 22,1% -> 10K,1%; device _RoweTel:RES-0805 -> AA-ipc-7351-resistor:RESISTOR_0402
- R21: value 0 Ohm -> 22,1%; device AA-ipc-7351-resistor:RESISTOR_0603 -> _RoweTel:RES-0805
- R22: value 22.1K,1% -> 10K,1%; device AA-ipc-7351-resistor:RESISTOR_0603 -> _RoweTel:RES-0805
- R23: value 10K,1% -> 2.2K,1%; device _RoweTel:RES-0805 -> AA-ipc-7351-resistor:RESISTOR_0402
- R24: value 47K,1% -> 22,1%
- R25: value 10K,1% -> 47K,1%
- R27: value 22,1% -> 10K,1%
- R28: value 22,1% -> 4.7K,1%
- R29: value 1.5K,1% -> 4.7K,1%; device AA-ipc-7351-resistor:RESISTOR_0402 -> _RoweTel:RES-0805
- R30: value 0 Ohm -> 1.5K,1%
- R31: value 0 Ohm -> 100,1%; device _RoweTel:RES-0805 -> AA-ipc-7351-resistor:RESISTOR_0603
- R33: value 2.2K,1/8W,5% -> 2.2K,1%; device _RoweTel:RES-0805 -> AA-ipc-7351-resistor:RESISTOR_0402
- R34: value 10K,1% -> 320,1%
- R35: value 330,1% -> 2.2K,1%; device _RoweTel:RES-0805 -> AA-ipc-7351-resistor:RESISTOR_0402
- R36: value 1.5K,1% -> 2.2K,1%; device _RoweTel:RES-0805 -> AA-ipc-7351-resistor:RESISTOR_0402
- R37: value 10K,1% -> 2.2K,1%
- R39: value 4.7,0.5W,1206 -> 500K,TrimPOT; device AA-ipc-7351-resistor:RESISTOR_1206 -> _RoweTel:POT3361
- R40: value 2.2K,1% -> 320,1%; device AA-ipc-7351-resistor:RESISTOR_0402 -> _RoweTel:RES-0805
- R41: value 2.2K,1% -> 0 Ohm; device AA-ipc-7351-resistor:RESISTOR_0402 -> AA-ipc-7351-resistor:RESISTOR_0603
- R42: value 500K,TrimPOT -> 1.5K,1%; device _RoweTel:POT3361 -> AA-ipc-7351-resistor:RESISTOR_0402
- R43: device _RoweTel:RES-0805 -> AA-ipc-7351-resistor:RESISTOR_0402
- R45: value 18K,1% -> 22.1K,1%; device _RoweTel:RES-0805 -> AA-ipc-7351-resistor:RESISTOR_0603
- R46: value 100K,POT -> 10K,1%; device _RoweTel:POT-3310C -> _RoweTel:RES-0805
- R47: value 18K,1% -> 2.2K,1/8W,5%
- R48: value 68K,1% -> 100K,POT; device _RoweTel:RES-0805 -> _RoweTel:POT-3310C
- R49: value 2.2K,1% -> 4.7,0.5W,1206; device _RoweTel:RES-0805 -> AA-ipc-7351-resistor:RESISTOR_1206
- R5: value 4.7K,1% -> 22,1%
- R50: value 10,1% -> 1K,1%; device AA-ipc-7351-resistor:RESISTOR_0603 -> _RoweTel:RES-0805
- R51: value 320,1% -> 124.0K,1%; device _RoweTel:RES-0805 -> AA-ipc-7351-resistor:RESISTOR_0402
- R52: value 1K,1% -> 22.1K,1%; device _RoweTel:RES-0805 -> AA-ipc-7351-resistor:RESISTOR_0402
- R53: value 2.2K,1% -> 10,1%; device AA-ipc-7351-resistor:RESISTOR_0402 -> AA-ipc-7351-resistor:RESISTOR_0603
- R54: value 0 Ohm -> 10K,1%
- R56: value 2.2K,1% -> 2.2K,1/8W,5%; device AA-ipc-7351-resistor:RESISTOR_0402 -> _RoweTel:RES-0805
- R57: value 470,1% -> 1K,1%; device AA-ipc-7351-resistor:RESISTOR_0402 -> _RoweTel:RES-0805
- R58: value 2.2K,1% -> 10,1%; device AA-ipc-7351-resistor:RESISTOR_0402 -> _RoweTel:RES-0805
- R59: value 330,1% -> 10K,1%
- R6: value 1K,1% -> 22,1%
- R60: value 3K,1% -> 2.2K,1%
- R61: value 4.7K,1% -> 10,1%
- R62: value 4.7K,1% -> 47,1%
- R64: value 10K,1% -> 470,1%
- R65: value 2.2K,1% -> 330,1%
- R67, R77: value 15,1% -> 2.2K,1%
- R68: value 2.2K,1% -> 15,1%
- R69: value 470,1% -> 15,1%
- R7, R8, R9: value 10K,1% -> 4.7K,1%
- R70: value 10,1% -> 2.2K,1%
- R71: value 47,1% -> 330,1%
- R72: value 330,1% -> 180,1%
- R73: value 680,1% -> 470,1%
- R75: value 2.2K,1% -> 47,1%
- R76: value 180,1% -> 10K,1%
- R78: value 2.2K,1% -> 18K,1%
- R79: value 470,1% -> 18K,1%
- R80: value 10,1% -> 10K,1%
- R81: value 47,1% -> 10K,1%
- R82: value 39K,1% -> 3K,1%
- R83: value 18K,1% -> 10K,1%
- R85, R91: value 3.3K,1% -> 10,1%
- R86: value 10,1% -> 3K,1%
- R87: value 10,1% -> 1K,1%
- R88: value 2.2K,1% -> 49.9,1%
- R89: value 100,1% -> 4.7K,1%
- R90: value 100,1% -> 2.2K,1%
- R92: value 150,1% -> 47,1%, DNL
- R93: value 3K,1% -> 330,1%
- R94: value 1K,1% -> 68K,1%
- R95: value 49.9,1% -> 10K,1%
- R96, R97: value 10,1% -> 0 Ohm
- R98: value 47,1%, DNL -> 0 Ohm
- R99: value 4.7K,1% -> 1K,1%
- SW1: value SW-LC2259 -> TS-02B; device _RoweTel:SW-LC2259 -> _RoweTel:TS-02B
- SW2: value TS-026 -> SW-LC2259; device _RoweTel:TS-026 -> _RoweTel:SW-LC2259
- SW3: value SW-LC2259EENP -> TS-026; device _RoweTel:SW-LC2259 -> _RoweTel:TS-026
- SW5: value TS-02B -> SW-LC2259EENP; device _RoweTel:TS-02B -> _RoweTel:SW-LC2259
- U10: value DNL -> LM386M-1; device _RoweTel:I2C-EEPROM-256K -> _RoweTel:LM386M-1
- U11: value L78MXX -> ADE-1; device _RoweTel:L78MXX -> _RoweTel:ADE-1
- U13: value ADE-1 -> LMV341; device _RoweTel:ADE-1 -> _RoweTel:LMV341
- U14: value SI570 -> SI5351A; device _RoweTel:SI570 -> _RoweTel:SI5351A
- U15: value SI5351A -> SI570; device _RoweTel:SI5351A -> _RoweTel:SI570
- U2: value L78MXX -> STMPS2141; device _RoweTel:L78MXX -> _RoweTel:STMPS2141
- U3: value STMPS2141 -> EMIF02-USB03F2; device _RoweTel:STMPS2141 -> AA-IC:EMIF02-USB03F2
- U4: value EMIF02-USB03F2 -> DNL; device AA-IC:EMIF02-USB03F2 -> _RoweTel:I2C-EEPROM-256K
- U5: value LMV341 -> L78MXX; device _RoweTel:LMV341 -> _RoweTel:L78MXX
- U6: value AP7215Y-33 -> L78MXX; device _RoweTel:AP7215Y -> _RoweTel:L78MXX
- U7: value SA612A -> LMV341; device _RoweTel:SA612A -> _RoweTel:LMV341
- U8: value LM386M-1 -> AP7215Y-33; device _RoweTel:LM386M-1 -> _RoweTel:AP7215Y
- U9: value LMV341 -> TPS54329E; device _RoweTel:LMV341 -> _RoweTel:TPS54329E
- XTAL2: value ECS-10.7-15B -> 25MHz,TXC,SMD; device _RoweTel:ECS-10.7-15B -> _RoweTel:XTAL-FY0800035
- renumbered C141 to C86, C142 to C85, C143 to C83, C166 to C46, CN8 to CN7, D13 to D9, L24 to L7, P14 to P2, P19 to P5
Connections:
- removed net N$129: J8.1
- net !BACK!: now also R27.1; no longer R8.1
- net !BOOT0!: now also R19.1; no longer R57.1
- net !EXT-PTT!: now also R23.2; no longer R56.2
- net !SELECT!: now also R22.1, SW3.1; no longer R7.1, SW2.1
- net !TEST!: now also R7.2; no longer R4.2
- net +12VRXENB: now also R54.1, U1A.PE5; no longer R34.1
- net +12VTXENB: now also R46.1, U1A.PE4; no longer R18.1
- net +5V: now also C26.1, C51.1, C54.1, FB16.2, FB17.1, FB19.2, FB4.1, R51.1, R55.2, U2.IN, U6.IN; no longer C108.1, C167.1, C7.1, FB10.2, FB14.2, FB15.1, FB8.1, R116.2, R127.1, U11.IN, U3.IN
- net +9V: now also C108.1, C109.1, C24.1, L15.2, R30.2, U5.OUT; no longer C38.1, C4.1, C41.1, L2.2, R36.2, U2.OUT
- net +VIN: now also C34.1, C56.1, P10.1, Q2.S, Q4.S, R40.2, R41.1, R47.2, R49.1, R56.2, SW5.2, SW5.3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; no longer C31.1, C63.1, P20.1, Q11.S, Q9.S, R117.2, R17.2, R21.1, R33.2, R39.1, SW3.2, SW3.3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
- net 1ST_LO: now also R96.1, R97.1, R98.1; no longer R105.1, R106.1, R107.1
- net 3V3: now also C1.1, C14.1, C15.1, C2.1, C29.1, C3.1, C5.1, C9.1, FB14.1, FB15.1, P1.1, R10.1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; no longer C16.1, C17.1, C18.1, C19.1, C20.1, C21.1, C52.1, C53.1, FB16.1, FB22.1, P13.1, R2.1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
- net A3V3: now also C38.1, C44.1, C45.1, FB1.1, FB9.2, R44.2, U13.!SHDN!, U13.V+, U7.!SHDN!, U7.V+, U8.OUT; no longer C22.1, C6.1, C65.1, FB21.2, FB7.1, R51.2, U5.!SHDN!, U5.V+, U6.OUT, U9.!SHDN!, U9.V+
- net AIN1: now also C13.1; no longer C56.1
- net AIN2: now also C10.1, P12.1, R42.1; no longer C55.1, P4.1, R29.1
- net AIN_PWR: now also C97.2, D10.K; no longer C26.2, D4.K
- net ANT_SMA: now also C100.1, C101.2, R94.2; no longer C147.1, C25.2, R48.2
- net BBAMP: now also C135.2, J14.1, L20.2; no longer C134.2, J7.1, L23.2
- net BOOT1: now also R11.2; no longer R6.2
- net DAC2_OUT: now also C48.1, P13.1, R13.2, R45.1; no longer C37.1, P3.1, R22.1, R54.2
- net DRIVER/PA_INPUT: now also C74.2, J10.1; no longer C137.2
- net GND: now also C104.2, C105.2, C106.2, C107.2, C108.2, C111.2, C112.2, C113.2, C114.2, C116.A, C125.1, C127.2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; no longer C100.2, C113.1, C116.2, C118.2, C119.2, C123.A, C129.1, C130.1, C134.1, C135.2, C138.2, C145.2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
- net LED-ERR: now also R4.1; no longer R16.1
- net LED-PTT: now also R2.1; no longer R13.1
- net LED-PWR: now also R1.1; no longer R12.1
- net LED-RT: now also R3.1; no longer R15.1
- net MISO: now also P8.1; no longer P11.1
- net MOSI: now also P9.1; no longer P12.1
- net N$1: now also C17.1; no longer C14.1
- net N$10: now also C19.1, R15.2; no longer C2.1, R14.2
- net N$100: now also C72.1, FB7.2, R78.2; no longer C116.1, FB19.2, R45.2
- net N$101: now also C126.1, Q16.E, R113.2; no longer C79.1, Q7.E, R84.2
- net N$102: now also C134.1, FB18.2, R117.2, R119.2, R120.2; no longer C78.1, FB9.2, R85.2, R87.2, R90.2
- net N$103: now also C127.1, R110.2, R112.2, R115.2; no longer C77.1, R82.2, R86.2, R88.2
- net N$104: now also J14.2, Q16.B, R110.1, R111.2; no longer J7.2, Q7.B, R82.1, R83.2
- net N$105: now also Q16.C, Q17.B, R112.1; no longer Q7.C, Q8.B, R88.1
- net N$106: now also C130.2, Q17.E, R117.1; no longer C82.2, Q8.E, R85.1
- net N$107: now also C129.1, FB18.1, R115.1; no longer C80.1, FB9.1, R86.1
- net N$108: now also C126.2, R114.2; no longer C79.2, R89.2
- net N$109: now also C130.1, R119.1; no longer C82.1, R90.1
- net N$11: now also C80.2, J11.2; no longer C139.2, J10.2
- net N$110: now also Q17.C, R118.2; no longer Q8.C, R91.2
- net N$111: now also C136.1, FB19.1, R120.1; no longer C81.1, FB10.1, R87.1
- net N$112: now also C79.2, J10.2, L4.1; no longer C87.2, J8.2, L9.1
- net N$113: now also C99.1, R92.1; no longer C95.1, R98.1
- net N$114: now also C98.1, FB12.1, R89.2; no longer C96.1, FB11.1, R99.2
- net N$115: now also C73.1, D6.A, FB7.1; no longer C117.1, D10.A, FB19.1
- net N$116: now also C73.2, FB10.1; no longer C117.2, FB20.1
- net N$117: now also C74.1, D7.A, FB8.2; no longer C137.1, D11.A, FB18.2
- net N$118: now also C102.2, C105.1, L14.1; no longer C93.1, C98.2, L15.1
- net N$119: now also C111.1, FB13.2, U15.OE, U15.VDD; no longer C43.1, FB16.2, U14.OE, U14.VDD
- net N$12: now also C7.1, FB1.2, R12.1; no longer C13.1, FB7.2, R10.1
- net N$120: now also C113.1, FB14.2, U14.VDDO; no longer C44.1, FB22.2, U15.VDDO
- net N$121: now also R96.2, U14.CLK1; no longer R105.2, U15.CLK1
- net N$122: now also R97.2, U14.CLK2; no longer R106.2, U15.CLK2
- net N$123: now also R98.2, U15.CLK+; no longer R107.2, U14.CLK+
- net N$124: now also R100.2, R99.2, U14.CLK0; no longer R102.2, R103.2, U15.CLK0
- net N$125: now also C75.1, FB8.1, R79.2; no longer C115.1, FB18.1, R47.2
- net N$126: now also C66.1, C67.2, C69.2, L3.1; no longer C112.2, C113.2, C114.1, L17.1
- net N$127: now also LED8.A, R44.1; no longer LED7.A, R51.1
- net N$128: now also R80.1, R83.1, U13.-IN; no longer R43.1, R9.1, U5.-IN
- net N$13: now also R13.1; no longer R54.1
- net N$130: now also C104.1, C106.1, L13.1, L15.1; no longer C29.1, C5.1, L11.1, L2.1
- net N$131: now also LED9.A, R50.1; no longer LED8.A, R52.1
- net N$132: now also R34.1; no longer R44.1
- net N$133: now also LED11.A, R57.1; no longer LED9.A, R100.1
- net N$134: now also R55.1; no longer R116.1
- net N$135: now also D6.C, D7.C, FB6.2, J8.2; no longer D10.C, D11.C, FB17.2, J11.2
- net N$136: now also C80.1, C82.1, L5.1; no longer C138.1, C139.1, L18.1
- net N$137: now also C89.2, L8.1; no longer C140.2, L19.1
- net N$138: now also LED7.A, R40.1; no longer LED11.A, R117.1
- net N$139: now also C88.2; no longer C144.2
- net N$14: now also R17.2, R19.2, SW2.1, SW2.4; no longer R1.2, R57.2, SW1.1, SW1.4
- net N$140: now also C120.1, Q15.C, R103.2, R105.2; no longer C118.1, Q17.C, R110.2, R111.2
- net N$141: now also C117.2, Q14.C, Q15.B, R105.1; no longer C121.2, Q17.B, Q18.C, R108.1
- net N$142: now also C122.1, FB16.1, R108.1; no longer C119.1, FB14.1, R110.1
- net N$143: now also C112.1, L17.2, XTAL3.1; no longer C120.1, L20.2, XTAL2.1
- net N$144: now also C115.1, XTAL4.2; no longer C122.1, XTAL2.2
- net N$145: now also C116.E, C117.1, L18.2, XTAL4.1; no longer C121.1, C123.E, L21.2, XTAL3.1
- net N$146: now also C118.1, Q14.B, R103.1, R104.2; no longer C124.1, Q18.B, R111.1, R112.2
- net N$147: now also C121.1, Q14.E, R106.2; no longer C125.1, Q18.E, R113.2
- net N$148: now also C119.1, Q15.E, R107.2; no longer C126.1, Q17.E, R109.2
- net N$149: now also C89.1, C92.1, D8.A, L10.1; no longer C140.1, C145.1, D12.A, L25.1
- net N$15: now also C20.1, CN2.C, D1.C, R20.2, R23.1; no longer C51.1, CN10.C, D7.C, R37.2, R56.1
- net N$151: now also C123.2, L19.1, U16.IN_A; no longer C127.2, L22.1, U7.IN_A
- net N$152: now also FB17.2, R116.2; no longer FB15.2, R115.2
- net N$153: now also C133.2, R116.1, U16.VIN; no longer C130.2, R115.1, U7.VIN
- net N$154: now also C128.2, U16.OSC_B; no longer C132.2, U7.OSC_B
- net N$156: now also C132.2, L20.1, U16.OUT_A; no longer C133.2, L23.1, U7.OUT_A
- net N$157: now also C96.1, L11.2; no longer C149.1, L26.2
- net N$158: now also C103.1, L11.1, R90.1, R95.2; no longer C148.1, L26.1, R23.2, R49.1
- net N$16: now also R1.2; no longer R12.2
- net N$169: now also C49.1, U9.VBST; no longer C107.1, U17.VBST
- net N$17: now also R2.2; no longer R13.2
- net N$170: now also C51.2, R51.2, R52.1, U9.VFB; no longer C108.2, R127.2, R128.1, U17.VFB
- net N$171: now also C47.1, U9.SS; no longer C109.1, U17.SS
- net N$172: now also U9.VREG5; no longer U17.VREG5
- net N$173: now also R43.2, U9.EN; no longer R129.2, U17.EN
- net N$18: now also R3.2; no longer R15.2
- net N$19: now also L12.2, R91.1; no longer L13.2, R97.1
- net N$2: now also C16.1, R14.2; no longer C24.1, R31.2
- net N$20: now also R4.2; no longer R16.2
- net N$21: now also C62.1, C64.1, C66.2, L2.1; no longer C110.1, C111.1, C114.2, L16.1
- net N$22: now also CN4.DP, R24.1, U3.D+IN; no longer CN2.DP, R28.1, U4.D+IN
- net N$23: now also CN4.DM, R21.1, U3.D-IN; no longer CN2.DM, R27.1, U4.D-IN
- net N$24: now also D4.A, FB3.2; no longer D2.A, FB5.2
- net N$25: now also C27.1, C28.1, R31.2, R33.1; no longer C33.1, C34.1, R11.2, R58.1
- net N$26: now also FB2.2, R31.1; no longer FB4.2, R11.1
- net N$27: now also C39.2, R39.1, R42.2, U7.OUT; no longer C54.2, R29.2, R42.1, U9.OUT
- net N$28: now also CN4.ID, R26.1, U3.ID; no longer CN2.ID, R30.1, U4.ID
- net N$3: now also C18.1; no longer C15.1
- net N$30: now also C88.1; no longer C144.1
- net N$31: now also R16.2, R18.1, U2.!EN!; no longer R25.1, R26.2, U3.!EN!
- net N$32: now also C102.1, L13.2, Q13.D; no longer C98.1, L11.2, Q14.D
- net N$33: now also C93.1, FB12.2, Q13.G, R92.2; no longer C94.1, FB11.2, Q14.G, R98.2
- net N$34: now also C48.2, R48.3; no longer C37.2, R46.3
- net N$35: now also C28.2, R35.1; no longer C33.2, R41.1
- net N$37: now also C100.2, C95.1, L10.2; no longer C146.1, C147.2, L25.2
- net N$38: now also C94.1, FB11.2, R89.1; no longer C97.1, FB6.2, R99.1
- net N$39: now also C50.1, R48.2, U10.+IN; no longer C57.1, R46.2, U8.+IN
- net N$399: now also C40.1, C41.1, C42.1, C43.1, R41.2, R43.1, U9.VIN; no longer C150.1, C164.1, C179.1, C36.1, R129.1, R21.2, U17.VIN
- net N$4: now also C76.1, C77.1, FB10.2, FB9.1; no longer C135.1, C136.1, FB20.2, FB21.1
- net N$40: now also C119.2, J13.1; no longer C126.2, J6.1
- net N$41: now also C39.1, R37.2, R39.2, R39.3; no longer C54.1, R42.2, R42.3, R53.2
- net N$42: now also Q1.C, Q2.G, R47.1; no longer Q10.C, Q9.G, R17.1
- net N$43: now also C53.2, R53.1; no longer C40.2, R50.1
- net N$44: now also C55.2, FB5.1; no longer C39.2, FB3.1
- net N$45: now also C30.1, C31.+, R33.2; no longer C32.+, C62.1, R58.2
- net N$46: now also C32.+, C33.2, R36.1, U7.+IN; no longer C58.2, C59.+, R40.1, U9.+IN
- net N$47: now also C114.1, FB15.2, U14.VDD; no longer C42.1, FB13.2, U15.VDD
- net N$48: now also C52.1, R49.2, U10.VS; no longer C60.1, R39.2, U8.VS
- net N$49: now also C123.1, C124.2, J13.2, R109.2; no longer C127.1, C128.2, J6.2, R114.2
- net N$5: now also C6.1, R12.2; no longer C10.1, R10.2
- net N$50: now also Q3.C, Q4.G, R56.1; no longer Q11.G, Q15.C, R33.1
- net N$51: now also C124.1, C125.2, L19.2, U16.IN_B; no longer C128.1, C129.2, L22.2, U7.IN_B
- net N$52: now also C110.1, J12.1, L16.2; no longer C100.1, J9.1, L14.2
- net N$53: now also Q1.B, R46.2; no longer Q10.B, R18.2
- net N$54: now also C36.1, C37.1, FB4.2, U8.IN; no longer C1.1, C103.1, FB8.2, U6.IN
- net N$55: now also Q3.B, R54.2; no longer Q15.B, R34.2
- net N$56: now also C62.2, J7.2; no longer C111.2, J12.2
- net N$57: now also C101.1, D10.A, R93.2; no longer C25.1, D4.A, R35.2
- net N$58: now also J7.1, U11.RF; no longer J12.1, U13.RF
- net N$59: now also C78.2, J11.1; no longer C27.2, J10.1
- net N$6: now also R6.2; no longer R20.2
- net N$60: now also CN6.D; no longer CN5.D
- net N$61: now also C78.1; no longer C27.1
- net N$62: now also D5.C, FB5.2, J5.2; no longer D3.C, FB3.2, J2.2
- net N$63: now also R30.1; no longer R36.1
- net N$64: now also J5.1; no longer J2.1
- net N$65: now also U14.XA, XTAL2.3; no longer U15.XA, XTAL5.3
- net N$66: now also Q6.C, Q8.B, R65.2; no longer Q1.C, Q2.B, R59.2
- net N$67: now also C61.1, Q10.C, Q8.C, R58.1, R59.2, R65.1; no longer C68.1, Q2.C, Q3.C, R59.1, R64.2, R70.1
- net N$68: now also Q10.B, Q8.E, R70.2; no longer Q2.E, Q3.B, R68.2
- net N$69: now also C59.1; no longer C28.1
- net N$7: now also R5.2; no longer R19.2
- net N$70: now also C81.1, Q11.E, R84.2; no longer C88.1, Q12.E, R92.2
- net N$71: now also C91.1, Q12.E, R88.2; no longer C90.1, Q13.E, R95.2
- net N$73: now also C84.1, L6.1, R81.2, R85.2; no longer C91.1, L10.1, R55.2, R96.2
- net N$74: now also C90.1, L9.1, R85.1, R86.2, R91.2; no longer C92.1, L12.1, R93.2, R96.1, R97.2
- net N$75: now also C87.1, Q12.B, R86.1, R87.2; no longer C89.1, Q13.B, R93.1, R94.2
- net N$76: now also CN6.C, D2.C, FB2.1; no longer CN5.C, D8.C, FB4.1
- net N$77: now also C25.1, CN5.1, D3.C, FB3.1, P11.1; no longer C30.1, CN3.1, D1.C, FB5.1, P21.1
- net N$78: now also C79.1, Q11.B, R81.1, R82.2; no longer C87.1, Q12.B, R55.1, R60.2
- net N$79: now also C69.1, J8.1; no longer C112.1, J11.1
- net N$8: now also C53.1, C55.1, U10.OUT; no longer C39.1, C40.1, U8.OUT
- net N$80: now also U14.XB, XTAL2.1; no longer U15.XB, XTAL5.1
- net N$81: now also D4.C, SW5.1, SW5.4; no longer D2.C, SW3.1, SW3.4
- net N$82: now also C87.2, L6.2, Q11.C; no longer C89.2, L10.2, Q12.C
- net N$83: now also C57.1, C59.2, Q6.B, R59.1, R60.2; no longer C28.2, C71.1, Q1.B, R64.1, R65.2
- net N$84: now also C93.2, L9.2, Q12.C; no longer C94.2, L12.2, Q13.C
- net N$85: now also C60.1, Q6.E; no longer C67.1, Q1.E
- net N$86: now also C60.2, R68.2; no longer C67.2, R67.2
- net N$87: now also R35.2, R37.1, U7.-IN; no longer R41.2, R53.1, U9.-IN
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Other:
- note added: "+5V"
- note added: "+9V"
- note added: "+VIN"
- note added: "3V3"
- note added: "A3V3"
- note added: "RX+12V"
- note added: "TX+12V"
- note removed: "to T/R switch"

Commit message: RESTORE .SCH, .BRD, .EPF & .LBR FILES, DUE TO SNAFU ON THIS END.(THANKS DAVID) RGB
Parts:
- removed P11: TPAD50, _Coherix:TPAD50
- added TP1: SCOPE_PAD, _RoweTel:SCOPE_PAD
- C41: value 100nF,25V -> 1nF,25V
- C46, C47: device ipc-7351-capacitor:CAPACITOR_0603 -> AA-ipc-7351-capacitor:CAPACITOR_0603
Connections:
- net GND: now also TP1.2
- net N$77: now also TP1.1; no longer P11.1
Changed lines of the file:
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@@
 <setting verticaltext="up"/>
 </settings>
-<grid distance="0.1" unitdist="inch" unit="inch" style="lines" multiple="1" display="no" altdistance="0.01" altunitdist="inch" altunit="inch"/>
+<grid distance="0.1" unitdist="inch" unit="inch" style="lines" multiple="1" display="yes" altdistance="0.01" altunitdist="inch" altunit="inch"/>
 <layers>
 <layer number="1" name="Top" color="4" fill="1" visible="no" active="no"/>
@@
 <part name="V143" library="A-SUPPLY2" deviceset="GND" device=""/>
 <part name="D2" library="_RoweTel" deviceset="PESD5ZX" device="" value="DNL"/>
-<part name="P11" library="_Coherix" deviceset="TPAD50" device=""/>
 <part name="U4" library="_RoweTel" deviceset="I2C-EEPROM-256K" device="" value="DNL"/>
 <part name="V145" library="A-SUPPLY2" deviceset="GND" device=""/>
@@
 <part name="V127" library="A-SUPPLY2" deviceset="GND" device=""/>
 <part name="V133" library="A-SUPPLY2" deviceset="GND" device=""/>
-<part name="C47" library="ipc-7351-capacitor" deviceset="CAPACITOR_" device="0603" value="8.2nF,25V"/>
+<part name="C47" library="AA-ipc-7351-capacitor" deviceset="CAPACITOR_" device="0603" value="8.2nF,25V"/>
 <part name="V134" library="A-SUPPLY2" deviceset="GND" device=""/>
 <part name="R43" library="AA-ipc-7351-resistor" deviceset="RESISTOR_" device="0402" value="10K,1%"/>
@@
 <part name="V135" library="A-SUPPLY2" deviceset="GND" device=""/>
 <part name="V144" library="A-SUPPLY2" deviceset="+5V" device=""/>
-<part name="C41" library="_RoweTel" deviceset="CAP-0805" device="" value="100nF,25V"/>
 <part name="V184" library="A-SUPPLY2" deviceset="GND" device=""/>
-<part name="C46" library="ipc-7351-capacitor" deviceset="CAPACITOR_" device="0603" value="470nF,25V"/>
+<part name="C46" library="AA-ipc-7351-capacitor" deviceset="CAPACITOR_" device="0603" value="470nF,25V"/>
 <part name="V185" library="A-SUPPLY2" deviceset="GND" device=""/>
 <part name="C54" library="AA-ipc-7351-capacitor" deviceset="CAPACITOR_" device="1210" value="22uF,25V,1210"/>
@@
 <part name="V102" library="A-SUPPLY2" deviceset="3V3" device=""/>
 <part name="V106" library="A-SUPPLY2" deviceset="GND" device=""/>
+<part name="C41" library="_RoweTel" deviceset="CAP-0805" device="" value="1nF,25V"/>
+<part name="TP1" library="_RoweTel" deviceset="SCOPE_PAD" device=""/>
+<part name="V108" library="A-SUPPLY2" deviceset="GND" device=""/>
 </parts>
 <sheets>
@@
 <attribute name="VALUE" x="66.04" y="207.518" size="1.4224" layer="96"/>
 </instance>
-<instance part="FB3" gate="G$1" x="60.96" y="106.68"/>
+<instance part="FB3" gate="G$1" x="60.96" y="106.68" smashed="yes">
+<attribute name="NAME" x="61.722" y="108.712" size="1.4224" layer="95" ratio="10"/>
+<attribute name="VALUE" x="58.42" y="102.743" size="1.4224" layer="96" ratio="10"/>
+</instance>
 <instance part="R41" gate="G$1" x="137.16" y="106.68" smashed="yes">
 <attribute name="NAME" x="134.62" y="111.76" size="1.4224" layer="95" ratio="9"/>
@@
 <attribute name="VALUE" x="45.72" y="198.12" size="1.4224" layer="96" ratio="10"/>
 </instance>
-<instance part="P11" gate="G$1" x="53.34" y="109.22" smashed="yes">
-<attribute name="NAME" x="55.372" y="113.538" size="1.4224" layer="95"/>
-</instance>
 <instance part="U5" gate="G$1" x="22.86" y="152.4" smashed="yes">
 <attribute name="NAME" x="15.24" y="162.56" size="1.4224" layer="95" ratio="10"/>
@@
 <attribute name="VALUE" x="274.955" y="96.393" size="1.4224" layer="96" ratio="9" rot="R270"/>
 </instance>
-<instance part="C41" gate="G$1" x="149.86" y="99.06" smashed="yes">
-<attribute name="NAME" x="149.86" y="116.84" size="1.4224" layer="95" ratio="9"/>
-<attribute name="VALUE" x="149.86" y="114.3" size="1.4224" layer="96" ratio="9"/>
-</instance>
 <instance part="V184" gate="GND" x="149.86" y="91.44" smashed="yes">
 <attribute name="VALUE" x="147.32" y="88.138" size="1.4224" layer="96" ratio="9"/>
@@
 <attribute name="VALUE" x="127" y="72.898" size="1.4224" layer="96" ratio="9"/>
 </instance>
+<instance part="C41" gate="G$1" x="149.86" y="99.06" smashed="yes">
+<attribute name="VALUE" x="149.86" y="114.3" size="1.4224" layer="96" ratio="10"/>
+<attribute name="NAME" x="149.86" y="116.84" size="1.4224" layer="95" ratio="10"/>
+</instance>
+<instance part="TP1" gate="G$1" x="53.34" y="114.3" smashed="yes" rot="R90">
+<attribute name="NAME" x="51.562" y="111.76" size="1.4224" layer="95" ratio="10" rot="R90"/>
+</instance>
+<instance part="V108" gate="GND" x="53.34" y="121.92" smashed="yes" rot="R180">
+<attribute name="VALUE" x="55.88" y="125.222" size="1.4224" layer="96" ratio="9" rot="R180"/>
+</instance>
 </instances>
 <busses>
@@
 </segment>
 <segment>
-<pinref part="C41" gate="G$1" pin="2"/>
 <pinref part="V184" gate="GND" pin="GND"/>
 <wire x1="149.86" y1="93.98" x2="149.86" y2="96.52" width="0.1524" layer="91"/>
+<pinref part="C41" gate="G$1" pin="2"/>
 </segment>
 <segment>
@@
 <pinref part="V98" gate="GND" pin="GND"/>
 </segment>
+<segment>
+<pinref part="TP1" gate="G$1" pin="2"/>
+<pinref part="V108" gate="GND" pin="GND"/>
+</segment>
 </net>
 <net name="N$25" class="0">
@@
 <pinref part="C25" gate="G$1" pin="1"/>
 <wire x1="53.34" y1="104.14" x2="53.34" y2="106.68" width="0.1524" layer="91"/>
-<pinref part="P11" gate="G$1" pin="1"/>
 <wire x1="53.34" y1="109.22" x2="53.34" y2="106.68" width="0.1524" layer="91"/>
 <junction x="53.34" y="106.68"/>
+<pinref part="TP1" gate="G$1" pin="1"/>
 </segment>
 </net>
@@
 <junction x="154.94" y="106.68"/>
 <wire x1="149.86" y1="106.68" x2="154.94" y2="106.68" width="0.1524" layer="91"/>
-<pinref part="C41" gate="G$1" pin="1"/>
 <wire x1="149.86" y1="101.6" x2="149.86" y2="106.68" width="0.1524" layer="91"/>
 <junction x="149.86" y="106.68"/>
@@
 <junction x="144.78" y="106.68"/>
 <pinref part="R41" gate="G$1" pin="2"/>
+<pinref part="C41" gate="G$1" pin="1"/>
 </segment>
 </net>
