File: sm2000/CAD/SM2000.brd (EAGLE design)
At the start: 160 x 100 mm, 400 parts, among them CN1 HDR100-3, CN10 ST-3509, CN11 HDR100-3, CN2 JS-MU3-002, CN3 DS-0518, CN5 ST-3509, CN8 ST-3509, J1 JMP-2PIN, J10 JMPR-2X2, J11 JMPR-2X2, J12 JMPR-2X2, J13 JMPR-2X2, J14 HDR100-5, J2 JMP-2PIN, J3 JMP-2PIN, J4 CONN-BOOM-XH-2A, J5 JMPR-2X2, J6 JMPR-2X2, J7 JMPR-2X2, J8 JMPR-2X2, J9 JMPR-2X2, P10 TPAD50, P11 TPAD50, P12 TPAD50, P13 TPAD50, P14 TPAD50, P16 TPAD50, P18 TPAD50, P19 TPAD50, P20 TPAD50, P21 TPAD50, P3 TPAD50, P4 TPAD50, P9 TPAD50, Q1 MMBT3904, Q10 MMBT3904, Q11 STR2P3LLH6, Q12 BRF92, Q13 BFQ19, Q14 RD01MUS2, Q15 MMBT3904, Q17 MMBT3904, Q18 MMBT3904, Q2 MMBT3904, Q3 MMBT3904, Q4 MMBT3904, Q5 MMBT3904, Q6 MMBT3904, Q7 MMBT3904, Q8 MMBT3906, Q9 STR2P3LLH6, SW1 SW-LC2259, SW2 TS-026, SW3 SW-LC2259EENP, SW4 TS-026, SW5 TS-02B, U1 STM32F405VGT6, U10 DNL, U11 L78MXX, U12 PGA-103+, U13 ADE-1, U14 SI570, U15 SI5351A, U17 TPS54329E, U2 L78MXX, U3 STMPS2141, U4 EMIF02-USB03F2, U5 LMV341, U6 AP7215Y-33, U7 SA612A, U8 LM386M-1, U9 LMV341, X1 BU-SMA-H

Commit message: Cleaned up schematic. Ran ERC with no errors. Started arranging parts on board. Have to add scope test points. A lot of parts to fit on PCB! RGB
Parts:
- removed C137, C147, C148, C149: 1nF,25V, _RoweTel:C0805
- removed C138, C141: 12pF,50V, _RoweTel:C0805
- removed C139, C140: 3.3pF,50V, _RoweTel:C0805
- removed C142: 0.5pF,50V, _RoweTel:C0805
- removed C143, C144: 2.2pF,50V, _RoweTel:C0805
- removed C145: 22pF,50V, _RoweTel:C0805
- removed C146: 22pF,25V, _RoweTel:C0805
- removed C150, C179: 22uF,25V, _RoweTel:C1210
- removed C164: 100nF,25V, _RoweTel:C0805
- removed C167: 22uF,25V,1210, AA-ipc-7351-capacitor:CAPC3225X168N
- removed CN10, CN8: ST-3509, _RoweTel:ST-3509
- removed CN11: HDR100-3, _Coherix:HDR100-3
- removed D11, D12, D13: BAR64-02V, _RoweTel:SC79_INFINEON
- removed FB20, FB21, FB22: FB0805, _RoweTel:FE0805
- removed L21: 9.2uH, _RoweTel:L-TDK-MLF2012
- removed L22: 5.2uH, _RoweTel:L-TDK-MLF2012
- removed L23: 15uH, _RoweTel:L-TDK-MLF2012
- removed L24: 260nH, rcl:0204/5
- removed L25: 53nH 3T 5mm ID, _RoweTel:L10X15
- removed L26: 220nH, _RoweTel:L10X15
- removed P16, P18, P20, P21: TPAD50, _Coherix:TPAD50
- removed Q18: MMBT3904, transistor:SOT23-EBC
- removed R127: 124.0K,1%, AA-ipc-7351-resistor:RESC1005X40AN
- removed R128: 22.1K,1%, AA-ipc-7351-resistor:RESC1005X40AN
- removed R129: 10K,1%, AA-ipc-7351-resistor:RESC1005X40AN
- removed SH4, SH5: SHUNT, _RoweTel:SHUNT
- removed U17: TPS54329E, _RoweTel:PSO-DDA
- removed XTAL5: 25MHz,TXC,SMD, _RoweTel:XTAL-FY0800035
- added C101: 1pF,50V, _RoweTel:C0805
- added C102, C106: 1nF,25V, _RoweTel:C0805
- added C104, C84: 0.1uF.25V, _RoweTel:C0805
- added C105: 33pF,50V, _RoweTel:C0805
- added C45, C61, C70: 100nF,25V, _RoweTel:C0805
- added C47: 8.2nF,25V, ipc-7351-capacitor:CAPC1608X92N
- added C48: 100nF,25V, AA-ipc-7351-capacitor:CAPC1005X60N
- added C50: 3.9nF,16V, _RoweTel:C0805
- added C64: 12pF.50V, _RoweTel:C0805
- added C66, C85: 0.5pF,50V, _RoweTel:C0805
- added C83: 2.2pF,50V, _RoweTel:C0805
- added C86: 12pF,50V, _RoweTel:C0805
- added CN4: JS-MU3-002, _RoweTel:JI-MU3-002
- added CN6, CN7: ST-3509, _RoweTel:ST-3509
- added D5: DNL, _RoweTel:SOD128
- added D6, D9: BAR64-02V, _RoweTel:SC79_INFINEON
- added FB1, FB12, FB2: FB0805, _RoweTel:FE0805
- added L3, L5, L8: 68nH, _RoweTel:L10X15
- added L4: 57nH, _RoweTel:L10X15
- added L6: 168nH, _RoweTel:L10X15
- added L7: 260nH, rcl:0204/5
- added P1, P6, P7, P8: TPAD50, _Coherix:TPAD50
- added Q16: MMBT3904, _RoweTel:SOT23
- added R118: 3.3K,1%, _RoweTel:R0805
- added R119: 100,1%, _RoweTel:R0805
- added R120: 10,1%, _RoweTel:R0805
- added U16: SA612A, _RoweTel:SO-08
- added XTAL4: ECS-10.7-15B, _RoweTel:HC49/S
- C1: value 22uF,25V -> 100nF,25V; device _RoweTel:C1210 -> _RoweTel:C0805
- C10: value 1uF,16V -> 1nF,25V
- C100: value 33pF,50V -> 1nF,25V
- C107: value 100nF,25V -> 47pF,50V; device AA-ipc-7351-capacitor:CAPC1005X60N -> _RoweTel:C0805
- C108: value 20pF,50V -> 0.1uF.25V; device AA-ipc-7351-capacitor:CAPC1005X60N -> _RoweTel:C0805
- C109: value 8.2nF,25V -> 100uF,25V,EL; device ipc-7351-capacitor:CAPC1608X92N -> _RoweTel:CAP-CHEMI-F80
- C110: value 12pF.50V -> 33pF,50V
- C111: value 3.3pF,50V -> 0.1uF,25V
- C112: value 3.3pF,50V -> 39pF,50V
- C113: value 12pF,50V -> 0.1uF,25V
- C114: value 0.5pF,50V -> 0.1uF,25V
- C115: value 1nF,25V -> 5.6pF,50V
- C116: value 1nF,25V -> 2-12pF; device _RoweTel:C0805 -> c-trimm:3008
- C117, C133, C134: value 1nF,25V -> 0.1uF,25V
- C119: value 10uF,25V,EL -> 0.1uF,25V; device _RoweTel:NICHICON-WJ-5 -> _RoweTel:C0805
- C12, C24: value 1uF,16V -> 100nF,25V
- C120: value 39pF,50V -> 0.1uF,25V
- C122: value 5.6pF,50V -> 10uF,25V,EL; device _RoweTel:C0805 -> _RoweTel:NICHICON-WJ-5
- C123: value 2-12pF -> 27pF,50V; device c-trimm:3008 -> _RoweTel:C0805
- C124: value 0.1uF,25V -> 150pF,50V
- C125: value 0.1uF,25V -> 0.1uF.25V
- C126: value 0.1uF,25V -> 10uF,25V,EL; device _RoweTel:C0805 -> _RoweTel:NICHICON-WJ-5
- C127: value 27pF,50V -> 0.1uF,25V
- C129: value 0.1uF.25V -> 10uF,25V,EL; device _RoweTel:C0805 -> _RoweTel:NICHICON-WJ-5
- C13, C72, C73, C74, C75, C76: value 100nF,25V -> 1nF,25V
- C130: value 1nF,25V -> 10uF,25V,EL; device _RoweTel:C0805 -> _RoweTel:NICHICON-WJ-5
- C131, C78: value 0.1uF,25V -> 1nF,25V
- C132: value 150pF,50V -> 1nF,25V
- C136: value 1uF,25V,EL -> 10uF,25V,EL; device _RoweTel:C1206-TANT -> _RoweTel:NICHICON-WJ-5
- C14, C35: value 2.2uF,16V -> 100nF,25V
- C15: value 2.2uF,16V -> 10nF,25V
- C16, C6: value 100nF,25V -> 1uF,16V
- C17: value 10nF,25V -> 2.2uF,16V
- C18: value 100nF,25V -> 2.2uF,16V
- C19, C21: value 10nF,25V -> 20pF,50V
- C2: value 20pF,50V -> 10nF,25V
- C22: value 100nF,25V -> 4.7uF,16V,TANT; device _RoweTel:C0805 -> _RoweTel:C1206-TANT
- C23: value 100nF,25V -> CAP-10UF-WJ5; device _RoweTel:C0805 -> _RoweTel:NICHICON-WJ-5
- C25: value 1pF,50V -> 10nF,25V
- C26: value 1nF,25V -> CAP-10UF-WJ5; device _RoweTel:C0805 -> _RoweTel:NICHICON-WJ-5
- C27: value 1nF,25V -> 1nF,25V,0402
- C28: value 100nF,25V -> 220nF,25V
- C29, C56: value 1nF,25V -> 100nF,25V
- C3: value 20pF,50V -> 100nF,25V
- C30: value 10nF,25V -> 100nF,25V
- C31: value CAP-10UF-WJ5 -> 100uF,6.3V,EL; device _RoweTel:NICHICON-WJ-5 -> _RoweTel:NICHICON-WX-6.3
- C33: value 220nF,25V -> 100nF,25V
- C34: value 1nF,25V,0402 -> 220uF,25V; device _RoweTel:C0805 -> _RoweTel:CAP-CHEMI-HA0
- C36: value 1nF,25V -> 22uF,25V; device _RoweTel:C0805 -> _RoweTel:C1210
- C37: value 100nF,25V -> 1nF,25V; device AA-ipc-7351-capacitor:CAPC1005X60N -> _RoweTel:C0805
- C38: value 100uF,25V,EL -> 2.2uF,16V; device _RoweTel:CAP-CHEMI-F80 -> _RoweTel:C0805
- C39: value 220uF,25V -> 100pF,50V; device _RoweTel:CAP-CHEMI-HA0 -> _RoweTel:C0805
- C40: value 47nF,25V -> 1nF,25V
- C41: value 0.1uF.25V -> 100nF,25V
- C42, C43: value 0.1uF,25V -> 22uF,25V; device _RoweTel:C0805 -> _RoweTel:C1210
- C44: value 0.1uF,25V -> 1uF,25V
- C49: device _RoweTel:C0805 -> AA-ipc-7351-capacitor:CAPC1005X60N
- C5: value 0.1uF.25V -> 10nF,25V
- C51: value 100nF,25V -> 20pF,50V; device _RoweTel:C0805 -> AA-ipc-7351-capacitor:CAPC1005X60N
- C52: value 100nF,25V -> 220uF,25V; device _RoweTel:C0805 -> _RoweTel:CAP-CHEMI-HA0
- C53: value 10nF,25V -> 47nF,25V
- C54: value 100pF,50V -> 22uF,25V,1210; device _RoweTel:C0805 -> AA-ipc-7351-capacitor:CAPC3225X168N
- C55: value 1nF,25V -> 220uF,25V; device _RoweTel:C0805 -> _RoweTel:CAP-CHEMI-HA0
- C57: value 3.9nF,16V -> 100nF,25V
- C59: value 100uF,6.3V,EL -> 100nF,25V; device _RoweTel:NICHICON-WX-6.3 -> _RoweTel:C0805
- C60, C63: value 220uF,25V -> 100nF,25V; device _RoweTel:CAP-CHEMI-HA0 -> _RoweTel:C0805
- C62, C69: value 100nF,25V -> 3.3pF,50V
- C65: value 1uF,25V -> 100nF,25V
- C67: value 100nF,25V -> 12pF,50V
- C7: value CAP-10UF-WJ5 -> 1uF,16V; device _RoweTel:NICHICON-WJ-5 -> _RoweTel:C0805
- C77: value 0.1uF,25V -> 1uF,25V,EL; device _RoweTel:C0805 -> _RoweTel:C1206-TANT
- C79: value 10uF,25V,EL -> 22pF,50V; device _RoweTel:NICHICON-WJ-5 -> _RoweTel:C0805
- C80: value 10uF,25V,EL -> 3.3pF,50V; device _RoweTel:NICHICON-WJ-5 -> _RoweTel:C0805
- C81: value 10uF,25V,EL -> 1nF,25V; device _RoweTel:NICHICON-WJ-5 -> _RoweTel:C0805
- C82: value 10uF,25V,EL -> 12pF,50V; device _RoweTel:NICHICON-WJ-5 -> _RoweTel:C0805
- C87: value 22pF,50V -> 5.6pF,50V
- C88: value 1nF,25V -> 2.2pF,50V
- C89: value 5.6pF,50V -> 3.3pF,50V
- C9: value 4.7uF,16V,TANT -> 10nF,25V; device _RoweTel:C1206-TANT -> _RoweTel:C0805
- C90: value 1nF,25V -> 0.1uF.25V
- C91, C97: value 0.1uF.25V -> 1nF,25V
- C92: value 0.1uF.25V -> 22pF,50V
- C93: value 33pF,50V -> 22pF,50V
- C94: value 22pF,50V -> 0.1uF.25V
- C95: value 1nF,25V -> 22pF,25V
- C99: value 47pF,50V -> 1nF,25V
- CN2: value JS-MU3-002 -> ST-3509; device _RoweTel:JI-MU3-002 -> _RoweTel:ST-3509
- CN3: value DS-0518 -> HDR100-3; device _RoweTel:DS-0518 -> _Coherix:HDR100-3
- CN5: value ST-3509 -> DS-0518; device _RoweTel:ST-3509 -> _RoweTel:DS-0518
- D1: value PTVS20VP1UP -> DNL; device _RoweTel:SOD128 -> _RoweTel:SOD523
- D10: value BAR64-02V -> BAT18; device _RoweTel:SC79_INFINEON -> _RoweTel:SOT23
- D2: value BAT60J -> DNL; device _RoweTel:SOD323R_INFINEON -> _RoweTel:SOD523
- D3: value DNL -> PTVS20VP1UP
- D4: value BAT18 -> BAT60J; device _RoweTel:SOT23 -> _RoweTel:SOD323R_INFINEON
- D7, D8: value DNL -> BAR64-02V; device _RoweTel:SOD523 -> _RoweTel:SC79_INFINEON
- J14: value HDR100-5 -> JMPR-2X2; device _RoweTel:HDR100-5 -> _RoweTel:JMPR-2X2X.1
- J2: value JMP-2PIN -> HDR100-5; device _Coherix:JMPR-2PIN -> _RoweTel:HDR100-5
- J5: value JMPR-2X2 -> JMP-2PIN; device _RoweTel:JMPR-2X2X.1 -> _Coherix:JMPR-2PIN
- L10: value 168nH -> 53nH 3T 5mm ID
- L11: value RFC -> 220nH; device _RoweTel:Z15/4 -> _RoweTel:L10X15
- L12: value 54nH -> RFC; device _RoweTel:L10X15 -> _RoweTel:Z15/4
- L15: value 57nH -> RFC; device _RoweTel:L10X15 -> _RoweTel:Z15/4
- L16: value 68nH -> 57nH
- L17: value 68nH -> 5.7uH; device _RoweTel:L10X15 -> _RoweTel:L-TDK-MLF2012
- L18: value 68nH -> 9.2uH; device _RoweTel:L10X15 -> _RoweTel:L-TDK-MLF2012
- L19: value 68nH -> 5.2uH; device _RoweTel:L10X15 -> _RoweTel:L-TDK-MLF2012
- L2: value RFC -> 68nH; device _RoweTel:Z15/4 -> _RoweTel:L10X15
- L20: value 5.7uH -> 15uH
- L9: value 57nH -> 54nH
- LED11: value SML-LX0603GW -> SML-LX0603YW
- LED8: value SML-LX0603SRW -> SML-LX0603GW
- LED9: value SML-LX0603YW -> SML-LX0603SRW
- Q11: value STR2P3LLH6 -> BRF92
- Q12: value BRF92 -> BFQ19; device _RoweTel:SOT23 -> _RoweTel:SOT89
- Q13: value BFQ19 -> RD01MUS2
- Q14: value RD01MUS2 -> MMBT3904; device _RoweTel:SOT89 -> transistor:SOT23-EBC
- Q15: device _RoweTel:SOT23 -> transistor:SOT23-EBC
- Q17: value MMBT3904 -> MMBT3906; device transistor:SOT23-EBC -> transistor-pnp:TO5
- Q2, Q4: value MMBT3904 -> STR2P3LLH6
- Q8: value MMBT3906 -> MMBT3904; device transistor-pnp:TO5 -> _RoweTel:SOT23
- Q9: value STR2P3LLH6 -> MMBT3904
- R1, R55, R74: value 10K,1% -> 680,1%
- R10: value 47,1% -> 4.7K,1%
- R102, R84: value 1K,1% -> 150,1%
- R103: value 1K,1% -> 33K,1%
- R104: value 150,1% -> 15K,1%
- R105: value 0 Ohm -> 3K,1%
- R106, R107: value 0 Ohm -> 1K,1%
- R108: value 3K,1% -> 10,1%
- R109: value 1K,1% -> 49.9,1%
- R11: value 100,1% -> 1K,1%; device AA-ipc-7351-resistor:RESC1608X55N -> _RoweTel:R0805
- R110: value 10,1% -> 39K,1%
- R111: value 33K,1% -> 18K,1%
- R112: value 15K,1% -> 2.2K,1%
- R114: value 49.9,1% -> 100,1%
- R115: value 150,1% -> 10,1%
- R116: value 680,1% -> 150,1%
- R117: value 320,1% -> 3.3K,1%
- R12: value 680,1% -> 47,1%
- R13, R16: value 680,1% -> 0 Ohm
- R14: value 220,1% -> 0 Ohm
- R15: value 680,1% -> 220,1%
- R17: value 2.2K,1/8W,5% -> 10K,1%
- R19: value 22,1% -> 470,1%; device _RoweTel:R0805 -> AA-ipc-7351-resistor:RESC1005X40AN
- R2, R3, R4: value 4.7K,1% -> 680,1%
- R20: value 22,1% -> 10K,1%; device _RoweTel:R0805 -> AA-ipc-7351-resistor:RESC1005X40AN
- R21: value 0 Ohm -> 22,1%; device AA-ipc-7351-resistor:RESC1608X55N -> _RoweTel:R0805
- R22: value 22.1K,1% -> 10K,1%; device AA-ipc-7351-resistor:RESC1608X55N -> _RoweTel:R0805
- R23: value 10K,1% -> 2.2K,1%; device _RoweTel:R0805 -> AA-ipc-7351-resistor:RESC1005X40AN
- R24: value 47K,1% -> 22,1%
- R25: value 10K,1% -> 47K,1%
- R27: value 22,1% -> 10K,1%
- R28: value 22,1% -> 4.7K,1%
- R29: value 1.5K,1% -> 4.7K,1%; device AA-ipc-7351-resistor:RESC1005X40AN -> _RoweTel:R0805
- R30: value 0 Ohm -> 1.5K,1%
- R31: value 0 Ohm -> 100,1%; device _RoweTel:R0805 -> AA-ipc-7351-resistor:RESC1608X55N
- R33: value 2.2K,1/8W,5% -> 2.2K,1%; device _RoweTel:R0805 -> AA-ipc-7351-resistor:RESC1005X40AN
- R34: value 10K,1% -> 320,1%
- R35: value 330,1% -> 2.2K,1%; device _RoweTel:R0805 -> AA-ipc-7351-resistor:RESC1005X40AN
- R36: value 1.5K,1% -> 2.2K,1%; device _RoweTel:R0805 -> AA-ipc-7351-resistor:RESC1005X40AN
- R37: value 10K,1% -> 2.2K,1%
- R39: value 4.7,0.5W,1206 -> 500K,TrimPOT; device AA-ipc-7351-resistor:RESC3115X70N -> _RoweTel:POT3361
- R40: value 2.2K,1% -> 320,1%; device AA-ipc-7351-resistor:RESC1005X40AN -> _RoweTel:R0805
- R41: value 2.2K,1% -> 0 Ohm; device AA-ipc-7351-resistor:RESC1005X40AN -> AA-ipc-7351-resistor:RESC1608X55N
- R42: value 500K,TrimPOT -> 1.5K,1%; device _RoweTel:POT3361 -> AA-ipc-7351-resistor:RESC1005X40AN
- R43: device _RoweTel:R0805 -> AA-ipc-7351-resistor:RESC1005X40AN
- R45: value 18K,1% -> 22.1K,1%; device _RoweTel:R0805 -> AA-ipc-7351-resistor:RESC1608X55N
- R46: value 100K,POT -> 10K,1%; device _RoweTel:POT-3310C -> _RoweTel:R0805
- R47: value 18K,1% -> 2.2K,1/8W,5%
- R48: value 68K,1% -> 100K,POT; device _RoweTel:R0805 -> _RoweTel:POT-3310C
- R49: value 2.2K,1% -> 4.7,0.5W,1206; device _RoweTel:R0805 -> AA-ipc-7351-resistor:RESC3115X70N
- R5: value 4.7K,1% -> 22,1%
- R50: value 10,1% -> 1K,1%; device AA-ipc-7351-resistor:RESC1608X55N -> _RoweTel:R0805
- R51: value 320,1% -> 124.0K,1%; device _RoweTel:R0805 -> AA-ipc-7351-resistor:RESC1005X40AN
- R52: value 1K,1% -> 22.1K,1%; device _RoweTel:R0805 -> AA-ipc-7351-resistor:RESC1005X40AN
- R53: value 2.2K,1% -> 10,1%; device AA-ipc-7351-resistor:RESC1005X40AN -> AA-ipc-7351-resistor:RESC1608X55N
- R54: value 0 Ohm -> 10K,1%
- R56: value 2.2K,1% -> 2.2K,1/8W,5%; device AA-ipc-7351-resistor:RESC1005X40AN -> _RoweTel:R0805
- R57: value 470,1% -> 1K,1%; device AA-ipc-7351-resistor:RESC1005X40AN -> _RoweTel:R0805
- R58: value 2.2K,1% -> 10,1%; device AA-ipc-7351-resistor:RESC1005X40AN -> _RoweTel:R0805
- R59: value 330,1% -> 10K,1%
- R6: value 1K,1% -> 22,1%
- R60: value 3K,1% -> 2.2K,1%
- R61: value 4.7K,1% -> 10,1%
- R62: value 4.7K,1% -> 47,1%
- R64: value 10K,1% -> 470,1%
- R65: value 2.2K,1% -> 330,1%
- R67, R77: value 15,1% -> 2.2K,1%
- R68: value 2.2K,1% -> 15,1%
- R69: value 470,1% -> 15,1%
- R7, R8, R9: value 10K,1% -> 4.7K,1%
- R70: value 10,1% -> 2.2K,1%
- R71: value 47,1% -> 330,1%
- R72: value 330,1% -> 180,1%
- R73: value 680,1% -> 470,1%
- R75: value 2.2K,1% -> 47,1%
- R76: value 180,1% -> 10K,1%
- R78: value 2.2K,1% -> 18K,1%
- R79: value 470,1% -> 18K,1%
- R80: value 10,1% -> 10K,1%
- R81: value 47,1% -> 10K,1%
- R82: value 39K,1% -> 3K,1%
- R83: value 18K,1% -> 10K,1%
- R85, R91: value 3.3K,1% -> 10,1%
- R86: value 10,1% -> 3K,1%
- R87: value 10,1% -> 1K,1%
- R88: value 2.2K,1% -> 49.9,1%
- R89: value 100,1% -> 4.7K,1%
- R90: value 100,1% -> 2.2K,1%
- R92: value 150,1% -> 47,1%, DNL
- R93: value 3K,1% -> 330,1%
- R94: value 1K,1% -> 68K,1%
- R95: value 49.9,1% -> 10K,1%
- R96, R97: value 10,1% -> 0 Ohm
- R98: value 47,1%, DNL -> 0 Ohm
- R99: value 4.7K,1% -> 1K,1%
- SW1: value SW-LC2259 -> TS-02B; device _RoweTel:SW-LC2259 -> _RoweTel:TS-02B
- SW2: value TS-026 -> SW-LC2259; device _RoweTel:TS-026 -> _RoweTel:SW-LC2259
- SW3: value SW-LC2259EENP -> TS-026; device _RoweTel:SW-LC2259 -> _RoweTel:TS-026
- SW5: value TS-02B -> SW-LC2259EENP; device _RoweTel:TS-02B -> _RoweTel:SW-LC2259
- U10: value DNL -> LM386M-1; device _RoweTel:SOIC8 -> _RoweTel:SO08
- U11: value L78MXX -> ADE-1; device _RoweTel:DPAK -> _RoweTel:ADE-1
- U13: value ADE-1 -> LMV341; device _RoweTel:ADE-1 -> _RoweTel:SOT23-6
- U14: value SI570 -> SI5351A; device _RoweTel:SI570 -> _RoweTel:MSOP10
- U15: value SI5351A -> SI570; device _RoweTel:MSOP10 -> _RoweTel:SI570
- U2: value L78MXX -> STMPS2141; device _RoweTel:DPAK -> _RoweTel:SOT23-5L
- U3: value STMPS2141 -> EMIF02-USB03F2; device _RoweTel:SOT23-5L -> AA-IC:ECOPACK-11
- U4: value EMIF02-USB03F2 -> DNL; device AA-IC:ECOPACK-11 -> _RoweTel:SOIC8
- U5: value LMV341 -> L78MXX; device _RoweTel:SOT23-6 -> _RoweTel:DPAK
- U6: value AP7215Y-33 -> L78MXX; device _RoweTel:SOT89 -> _RoweTel:DPAK
- U7: value SA612A -> LMV341; device _RoweTel:SO-08 -> _RoweTel:SOT23-6
- U8: value LM386M-1 -> AP7215Y-33; device _RoweTel:SO08 -> _RoweTel:SOT89
- U9: value LMV341 -> TPS54329E; device _RoweTel:SOT23-6 -> _RoweTel:PSO-DDA
- XTAL2: value ECS-10.7-15B -> 25MHz,TXC,SMD; device _RoweTel:HC49/S -> _RoweTel:XTAL-FY0800035
- moved R55 322.3 mm to (145.0, -10.0)
- moved Q13 300.3 mm to (111.5, -20.0)
- moved U15 284.9 mm to (52.5, -32.0)
- moved U5 267.8 mm to (98.0, -22.0)
- moved J2 255.5 mm to (146.5, -19.0)
- moved C25 251.8 mm to (22.0, 86.5)
- moved D4 249.4 mm to (22.8, 79.2)
- moved C42 244.6 mm to (45.6, 97.1), turned to 180 degrees
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- renumbered C166 to C46, P14 to P2, P19 to P5
Connections:
- removed net N$129: J8.1
- net !BACK!: now also R27.1; no longer R8.1
- net !BOOT0!: now also R19.1; no longer R57.1
- net !EXT-PTT!: now also R23.2; no longer R56.2
- net !SELECT!: now also R22.1, SW3.1; no longer R7.1, SW2.1
- net !TEST!: now also R7.2; no longer R4.2
- net +12VRXENB: now also R54.1, U1.4; no longer R34.1
- net +12VTXENB: now also R46.1, U1.3; no longer R18.1
- net +5V: now also C26.1, C51.1, C54.1, FB16.2, FB17.1, FB19.2, FB4.1, R51.1, R55.2, U2.5, U6.1; no longer C108.1, C167.1, C7.1, FB10.2, FB14.2, FB15.1, FB8.1, R116.2, R127.1, U11.1, U3.5
- net +9V: now also C108.1, C109.1, C24.1, L15.2, R30.2, U5.3; no longer C38.1, C4.1, C41.1, L2.2, R36.2, U2.3
- net +VIN: now also C34.1, C56.1, P10.1, Q2.2, Q4.2, R40.2, R41.1, R47.2, R49.1, R56.2, SW5.2, SW5.3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; no longer C31.1, C63.1, P20.1, Q11.2, Q9.2, R117.2, R17.2, R21.1, R33.2, R39.1, SW3.2, SW3.3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
- net 1ST_LO: now also R96.1, R97.1, R98.1; no longer R105.1, R106.1, R107.1
- net 3V3: now also C1.1, C14.1, C15.1, C2.1, C29.1, C3.1, C5.1, C9.1, FB14.1, FB15.1, P1.1, R10.1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; no longer C16.1, C17.1, C18.1, C19.1, C20.1, C21.1, C52.1, C53.1, FB16.1, FB22.1, P13.1, R2.1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
- net A3V3: now also C38.1, C44.1, C45.1, FB1.1, FB9.2, R44.2, U13.5, U13.6, U7.5, U7.6, U8.3; no longer C22.1, C6.1, C65.1, FB21.2, FB7.1, R51.2, U5.5, U5.6, U6.3, U9.5, U9.6
- net AIN1: now also C13.1; no longer C56.1
- net AIN2: now also C10.1, P12.1, R42.1; no longer C55.1, P4.1, R29.1
- net AIN_PWR: now also C97.2, D10.1; no longer C26.2, D4.1
- net ANT_SMA: now also C100.1, C101.2, R94.2; no longer C147.1, C25.2, R48.2
- net BBAMP: now also C135.2, J14.1, L20.P$2; no longer C134.2, J7.1, L23.P$2
- net BOOT1: now also R11.2; no longer R6.2
- net DAC2_OUT: now also C48.1, P13.1, R13.2, R45.1; no longer C37.1, P3.1, R22.1, R54.2
- net DRIVER/PA_INPUT: now also C74.2, J10.1; no longer C137.2
- net GND: now also C104.2, C105.2, C106.2, C107.2, C108.2, C111.2, C112.2, C113.2, C114.2, C116.-, C125.1, C127.2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; no longer C100.2, C113.1, C116.2, C118.2, C119.2, C123.-, C129.1, C130.1, C134.1, C135.2, C138.2, C141.1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
- net LED-ERR: now also R4.1; no longer R16.1
- net LED-PTT: now also R2.1; no longer R13.1
- net LED-PWR: now also R1.1; no longer R12.1
- net LED-RT: now also R3.1; no longer R15.1
- net MISO: now also P8.1; no longer P11.1
- net MOSI: now also P9.1; no longer P12.1
- net N$1: now also C17.1; no longer C14.1
- net N$10: now also C19.1, R15.2; no longer C2.1, R14.2
- net N$100: now also C72.1, FB7.2, R78.2; no longer C116.1, FB19.2, R45.2
- net N$101: now also C126.1, Q16.2, R113.2; no longer C79.1, Q7.2, R84.2
- net N$102: now also C134.1, FB18.2, R117.2, R119.2, R120.2; no longer C78.1, FB9.2, R85.2, R87.2, R90.2
- net N$103: now also C127.1, R110.2, R112.2, R115.2; no longer C77.1, R82.2, R86.2, R88.2
- net N$104: now also J14.2, Q16.1, R110.1, R111.2; no longer J7.2, Q7.1, R82.1, R83.2
- net N$105: now also Q16.3, Q17.2, R112.1; no longer Q7.3, Q8.2, R88.1
- net N$106: now also C130.2, Q17.1, R117.1; no longer C82.2, Q8.1, R85.1
- net N$107: now also C129.1, FB18.1, R115.1; no longer C80.1, FB9.1, R86.1
- net N$108: now also C126.2, R114.2; no longer C79.2, R89.2
- net N$109: now also C130.1, R119.1; no longer C82.1, R90.1
- net N$11: now also C80.2, J11.2; no longer C139.2, J10.2
- net N$110: now also Q17.3, R118.2; no longer Q8.3, R91.2
- net N$111: now also C136.1, FB19.1, R120.1; no longer C81.1, FB10.1, R87.1
- net N$112: now also C79.2, J10.2, L4.1; no longer C87.2, J8.2, L9.1
- net N$113: now also C99.1, R92.1; no longer C95.1, R98.1
- net N$114: now also C98.1, FB12.1, R89.2; no longer C96.1, FB11.1, R99.2
- net N$115: now also C73.1, D6.A, FB7.1; no longer C117.1, D10.A, FB19.1
- net N$116: now also C73.2, FB10.1; no longer C117.2, FB20.1
- net N$117: now also C74.1, D7.A, FB8.2; no longer C137.1, D11.A, FB18.2
- net N$118: now also C102.2, C105.1, L14.1; no longer C93.1, C98.2, L15.1
- net N$119: now also C111.1, FB13.2, U15.2, U15.6; no longer C43.1, FB16.2, U14.2, U14.6
- net N$12: now also C7.1, FB1.2, R12.1; no longer C13.1, FB7.2, R10.1
- net N$120: now also C113.1, FB14.2, U14.7; no longer C44.1, FB22.2, U15.7
- net N$121: now also R96.2, U14.9; no longer R105.2, U15.9
- net N$122: now also R97.2, U14.6; no longer R106.2, U15.6
- net N$123: now also R98.2, U15.4; no longer R107.2, U14.4
- net N$124: now also R100.2, R99.2, U14.10; no longer R102.2, R103.2, U15.10
- net N$125: now also C75.1, FB8.1, R79.2; no longer C115.1, FB18.1, R47.2
- net N$126: now also C66.1, C67.2, C69.2, L3.1; no longer C112.2, C113.2, C114.1, L17.1
- net N$127: now also LED8.A, R44.1; no longer LED7.A, R51.1
- net N$128: now also R80.1, R83.1, U13.3; no longer R43.1, R9.1, U5.3
- net N$13: now also R13.1; no longer R54.1
- net N$130: now also C104.1, C106.1, L13.1, L15.1; no longer C29.1, C5.1, L11.1, L2.1
- net N$131: now also LED9.A, R50.1; no longer LED8.A, R52.1
- net N$132: now also R34.1; no longer R44.1
- net N$133: now also LED11.A, R57.1; no longer LED9.A, R100.1
- net N$134: now also R55.1; no longer R116.1
- net N$135: now also D6.C, D7.C, FB6.2, J8.2; no longer D10.C, D11.C, FB17.2, J11.2
- net N$136: now also C80.1, C82.1, C85.2, L5.1; no longer C138.1, C139.1, C142.2, L18.1
- net N$137: now also C85.1, C86.2, C89.2, L8.1; no longer C140.2, C141.2, C142.1, L19.1
- net N$138: now also LED7.A, R40.1; no longer LED11.A, R117.1
- net N$139: now also C83.1, C88.2, L7.1; no longer C143.1, C144.2, L24.1
- net N$14: now also R17.2, R19.2, SW2.1, SW2.4; no longer R1.2, R57.2, SW1.1, SW1.4
- net N$140: now also C120.1, Q15.C, R103.2, R105.2; no longer C118.1, Q17.C, R110.2, R111.2
- net N$141: now also C117.2, Q14.C, Q15.B, R105.1; no longer C121.2, Q17.B, Q18.C, R108.1
- net N$142: now also C122.1, FB16.1, R108.1; no longer C119.1, FB14.1, R110.1
- net N$143: now also C112.1, L17.P$2, XTAL3.1; no longer C120.1, L20.P$2, XTAL2.1
- net N$144: now also C115.1, XTAL4.2; no longer C122.1, XTAL2.2
- net N$145: now also C116.+, C117.1, L18.P$2, XTAL4.1; no longer C121.1, C123.+, L21.P$2, XTAL3.1
- net N$146: now also C118.1, Q14.B, R103.1, R104.2; no longer C124.1, Q18.B, R111.1, R112.2
- net N$147: now also C121.1, Q14.E, R106.2; no longer C125.1, Q18.E, R113.2
- net N$148: now also C119.1, Q15.E, R107.2; no longer C126.1, Q17.E, R109.2
- net N$149: now also C89.1, C92.1, D8.A, L10.1; no longer C140.1, C145.1, D12.A, L25.1
- net N$15: now also C20.1, CN2.C, D1.C, R20.2, R23.1; no longer C51.1, CN10.C, D7.C, R37.2, R56.1
- net N$151: now also C123.2, L19.P$1, U16.1; no longer C127.2, L22.P$1, U7.1
- net N$152: now also FB17.2, R116.2; no longer FB15.2, R115.2
- net N$153: now also C133.2, R116.1, U16.8; no longer C130.2, R115.1, U7.8
- net N$154: now also C128.2, U16.6; no longer C132.2, U7.6
- net N$156: now also C132.2, L20.P$1, U16.4; no longer C133.2, L23.P$1, U7.4
- net N$157: now also C96.1, D9.A, L11.2; no longer C149.1, D13.A, L26.2
- net N$158: now also C103.1, L11.1, R90.1, R95.2; no longer C148.1, L26.1, R23.2, R49.1
- net N$16: now also R1.2; no longer R12.2
- net N$169: now also C49.1, U9.1; no longer C107.1, U17.1
- net N$17: now also R2.2; no longer R13.2
- net N$170: now also C51.2, R51.2, R52.1, U9.5; no longer C108.2, R127.2, R128.1, U17.5
- net N$171: now also C47.1, U9.8; no longer C109.1, U17.8
- net N$172: now also U9.6; no longer U17.6
- net N$173: now also R43.2, U9.7; no longer R129.2, U17.7
- net N$18: now also R3.2; no longer R15.2
- net N$19: now also L12.2, R91.1; no longer L13.2, R97.1
- net N$2: now also C16.1, R14.2; no longer C24.1, R31.2
- net N$20: now also R4.2; no longer R16.2
- net N$21: now also C62.1, C64.1, C66.2, L2.1; no longer C110.1, C111.1, C114.2, L16.1
- net N$22: now also CN4.3, R24.1, U3.C1; no longer CN2.3, R28.1, U4.C1
- net N$23: now also CN4.2, R21.1, U3.D1; no longer CN2.2, R27.1, U4.D1
- net N$24: now also D4.A, FB3.2; no longer D2.A, FB5.2
- net N$25: now also C27.1, C28.1, R31.2, R33.1; no longer C33.1, C34.1, R11.2, R58.1
- net N$26: now also FB2.2, R31.1; no longer FB4.2, R11.1
- net N$27: now also C39.2, R39.1, R42.2, U7.4; no longer C54.2, R29.2, R42.1, U9.4
- net N$28: now also CN4.4, R26.1, U3.A3; no longer CN2.4, R30.1, U4.A3
- net N$3: now also C18.1; no longer C15.1
- net N$30: now also C88.1; no longer C144.1
- net N$31: now also R16.2, R18.1, U2.4; no longer R25.1, R26.2, U3.4
- net N$32: now also C102.1, L13.2, Q13.3; no longer C98.1, L11.2, Q14.3
- net N$33: now also C93.1, FB12.2, Q13.1, R92.2; no longer C94.1, FB11.2, Q14.1, R98.2
- net N$34: now also C48.2, R48.3; no longer C37.2, R46.3
- net N$35: now also C28.2, R35.1; no longer C33.2, R41.1
- net N$36: now also C83.2; no longer C143.2
- net N$37: now also C100.2, C95.1, D9.C, L10.2; no longer C146.1, C147.2, D13.C, L25.2
- net N$38: now also C94.1, FB11.2, R89.1; no longer C97.1, FB6.2, R99.1
- net N$39: now also C50.1, R48.2, U10.3; no longer C57.1, R46.2, U8.3
- net N$399: now also C40.1, C41.1, C42.1, C43.1, R41.2, R43.1, U9.2; no longer C150.1, C164.1, C179.1, C36.1, R129.1, R21.2, U17.2
- net N$4: now also C76.1, C77.1, FB10.2, FB9.1; no longer C135.1, C136.1, FB20.2, FB21.1
- net N$40: now also C119.2, J13.1; no longer C126.2, J6.1
- net N$41: now also C39.1, R37.2, R39.2, R39.3; no longer C54.1, R42.2, R42.3, R53.2
- net N$42: now also Q1.3, Q2.1, R47.1; no longer Q10.3, Q9.1, R17.1
- net N$43: now also C53.2, R53.1; no longer C40.2, R50.1
- net N$44: now also C55.2, FB5.1; no longer C39.2, FB3.1
- net N$45: now also C30.1, C31.1, R33.2; no longer C32.1, C62.1, R58.2
- net N$46: now also C32.1, C33.2, R36.1, U7.1; no longer C58.2, C59.1, R40.1, U9.1
- net N$47: now also C114.1, FB15.2, U14.1; no longer C42.1, FB13.2, U15.1
- net N$48: now also C52.1, R49.2, U10.6; no longer C60.1, R39.2, U8.6
- net N$49: now also C123.1, C124.2, J13.2, R109.2; no longer C127.1, C128.2, J6.2, R114.2
- net N$5: now also C6.1, R12.2; no longer C10.1, R10.2
- net N$50: now also Q3.3, Q4.1, R56.1; no longer Q11.1, Q15.3, R33.1
- net N$51: now also C124.1, C125.2, L19.P$2, U16.2; no longer C128.1, C129.2, L22.P$2, U7.2
- net N$52: now also C110.1, J12.1, L16.2; no longer C100.1, J9.1, L14.2
- net N$53: now also Q1.1, R46.2; no longer Q10.1, R18.2
- net N$54: now also C36.1, C37.1, FB4.2, U8.2; no longer C1.1, C103.1, FB8.2, U6.2
- net N$55: now also Q3.1, R54.2; no longer Q15.1, R34.2
- net N$56: now also C62.2, J7.2; no longer C111.2, J12.2
- net N$57: now also C101.1, D10.3, R93.2; no longer C25.1, D4.3, R35.2
- net N$58: now also J7.1, U11.3; no longer J12.1, U13.3
- net N$59: now also C78.2, J11.1; no longer C27.2, J10.1
- net N$6: now also R6.2; no longer R20.2
- net N$60: now also CN6.D; no longer CN5.D
- net N$61: now also C78.1; no longer C27.1
- net N$62: now also CN7.C, D5.C, FB5.2, J5.2; no longer CN8.C, D3.C, FB3.2, J2.2
- net N$63: now also R30.1; no longer R36.1
- net N$64: now also CN7.B, J5.1; no longer CN8.B, J2.1
- net N$65: now also U14.2, XTAL2.3; no longer U15.2, XTAL5.3
- net N$66: now also Q6.3, Q8.1, R65.2; no longer Q1.3, Q2.1, R59.2
- net N$67: now also C61.1, Q10.3, Q8.3, R58.1, R59.2, R65.1; no longer C68.1, Q2.3, Q3.3, R59.1, R64.2, R70.1
- net N$68: now also Q10.1, Q8.2, R70.2; no longer Q2.2, Q3.1, R68.2
- net N$69: now also C59.1; no longer C28.1
- net N$7: now also R5.2; no longer R19.2
- net N$70: now also C81.1, Q11.2, R84.2; no longer C88.1, Q12.2, R92.2
- net N$71: now also C91.1, Q12.3, R88.2; no longer C90.1, Q13.3, R95.2
- net N$72: now also CN7.D; no longer CN8.D
- net N$73: now also C84.1, L6.1, R81.2, R85.2; no longer C91.1, L10.1, R55.2, R96.2
- net N$74: now also C90.1, L9.1, R85.1, R86.2, R91.2; no longer C92.1, L12.1, R93.2, R96.1, R97.2
- net N$75: now also C87.1, Q12.1, R86.1, R87.2; no longer C89.1, Q13.1, R93.1, R94.2
- net N$76: now also CN6.C, D2.C, FB2.1; no longer CN5.C, D8.C, FB4.1
- net N$77: now also C25.1, CN5.1, D3.C, FB3.1, P11.1; no longer C30.1, CN3.1, D1.C, FB5.1, P21.1
- net N$78: now also C79.1, Q11.1, R81.1, R82.2; no longer C87.1, Q12.1, R55.1, R60.2
- net N$79: now also C69.1, J8.1; no longer C112.1, J11.1
- net N$8: now also C53.1, C55.1, U10.5; no longer C39.1, C40.1, U8.5
- net N$80: now also U14.3, XTAL2.1; no longer U15.3, XTAL5.1
- net N$81: now also D4.C, SW5.1, SW5.4; no longer D2.C, SW3.1, SW3.4
- net N$82: now also C87.2, L6.2, Q11.3; no longer C89.2, L10.2, Q12.3
- net N$83: now also C57.1, C59.2, Q6.1, R59.1, R60.2; no longer C28.2, C71.1, Q1.1, R64.1, R65.2
- net N$84: now also C93.2, L9.2, Q12.2, Q12.2.1; no longer C94.2, L12.2, Q13.2, Q13.2.1
- net N$85: now also C60.1, Q6.2; no longer C67.1, Q1.2
- net N$86: now also C60.2, R68.2; no longer C67.2, R67.2
- net N$87: now also R35.2, R37.1, U7.3; no longer R41.2, R53.1, U9.3
- net N$88: now also Q10.2, R73.2, R75.1; no longer Q3.2, R69.2, R71.1
- net N$89: now also C70.2, R75.2; no longer C69.2, R71.2
- net N$9: now also C107.1, L14.2, L16.1; no longer C99.1, L14.1, L15.2
- net N$90: now also J6.2, U11.5; no longer J13.2, U13.5
- net N$91: now also Q7.1, Q9.3, R71.2, R74.2; no longer Q4.3, Q5.1, R72.2, R73.2
- net N$92: now also C63.1, Q7.3, R61.2, R71.1, R76.2; no longer C74.1, Q6.3, R72.1, R74.2, R80.2
- net N$93: now also Q5.1, Q7.2, R67.2; no longer Q5.2, Q6.1, R78.2
- net N$94: now also C68.1, R74.1; no longer C72.1, R73.1
- net N$95: now also C68.2, C71.1, Q9.1, R76.1, R77.2; no longer C72.2, C76.1, Q4.1, R74.1, R75.2
- net N$96: now also C65.1, Q9.2, R72.2; no longer C73.1, Q4.2, R76.2
- net N$97: now also C65.2, R69.2; no longer C73.2, R77.2
- net N$98: now also Q5.2, R62.1, R64.2; no longer Q6.2, R79.2, R81.1
- net N$99: now also C58.2, R62.2; no longer C75.2, R81.2
- net NRST: now also C4.1, R8.2, SW1.3, SW1.4; no longer C49.1, R3.2, SW5.3, SW5.4
- net NSS: now also P6.1; no longer P9.1
- net OSC_IN: now also C21.1; no longer C3.1
- net OSC_OUT: now also R15.1; no longer R14.1
- net OTG_DM: now also R21.2, U3.D3; no longer R27.2, U4.D3
- net OTG_DP: now also R24.2, U3.C3; no longer R28.2, U4.C3
- net OTG_ID: now also R26.2; no longer R30.2
- net OTG_OVR_CUR: now also R25.2, U2.3; no longer R24.2, U3.3
- net OTG_PWR_ON: now also R16.1; no longer R26.1
- net PA_OUTPUT: now also C96.2, J12.2; no longer C149.2, J9.2
- net PE0: now also J2.2; no longer J14.2
- net PE1: now also J2.3; no longer J14.3
- net PE2: now also J2.4; no longer J14.4
- net PE3: now also J2.5; no longer J14.5
- net RX+12V: now also Q2.3, R50.2, R58.2, R78.1; no longer Q9.3, R45.1, R52.2, R70.2
- net RX-2ND-LO: now also R100.1, R102.1; no longer R101.1, R103.1
- net SCK: now also P7.1; no longer P10.1
- net SCL3: now also R29.2, U14.4, U15.8, U4.6; no longer R62.2, U10.6, U14.8, U15.4
- net SDA3: now also R28.2, U14.5, U15.7, U4.5; no longer R61.2, U10.5, U14.7, U15.5
- net SW: now also C49.2, U9.3; no longer C107.2, U17.3
- net SWCLK: now also R5.1; no longer R19.1
- net SWDIO: now also R6.1; no longer R20.1
- net TIAIN: now also C57.2, C58.1, J6.1; no longer C71.2, C75.1, J13.1
- net TIAOUT: now also J9.2, L17.P$1; no longer J5.2, L20.P$1
- net TIA_OUT: now also C70.1, C71.2, J9.1; no longer C69.1, C76.2, J5.1
- net TX+12V: now also L12.1, Q4.3, R57.2, R61.1, R79.1, R90.2; no longer L13.1, Q11.3, R100.2, R47.1, R49.2, R80.1
- net TX-2ND-LO: now also R101.1, R99.1; no longer R102.1, R104.1
- net TX2NDLO: now also C121.2, C128.1; no longer C125.2, C132.1
- net TX_DAC: now also C118.2, U1.32; no longer C124.2
- net USART3_RX: now also CN3.3, R9.2; no longer CN11.3, R2.2
- net USART3_TX: now also CN3.1, R10.2; no longer CN11.1, R5.2
- net VBUS: now also C22.1, CN4.1, U2.1, U3.B3; no longer C9.1, CN2.1, U3.1, U4.B3
- net VGG: now also FB11.1, R83.2, U13.4; no longer FB6.1, R9.2, U5.4
- net VGG_DAC: now also U1.54, U13.1; no longer U5.1

Commit message: RESTORE .SCH, .BRD, .EPF & .LBR FILES, DUE TO SNAFU ON THIS END.(THANKS DAVID) RGB
Parts:
- removed P11: TPAD50, _Coherix:TPAD50
- added TP1: SCOPE_PAD, _RoweTel:SCOPE_PAD
- C41: value 100nF,25V -> 1nF,25V
- C46, C47: device ipc-7351-capacitor:CAPC1608X92N -> AA-ipc-7351-capacitor:CAPC1608X92N
- moved CN4 149.5 mm to (6.32, 25.3), turned to 90 degrees
- moved C54 135.7 mm to (63.3, 94.4), turned to 180 degrees
- moved LED10 131.2 mm to (69.0, 93.5)
- moved R55 131.2 mm to (69.0, 97.0)
- moved C49 119.4 mm to (62.6, 91.0)
- moved C51 117.1 mm to (62.6, 88.5)
- moved R51 113.8 mm to (62.6, 83.5)
- moved R52 113.2 mm to (62.6, 86.0)
- moved C46 110.8 mm to (66.1, 83.5)
- moved C47 110.8 mm to (66.1, 86.5)
- moved SW2 104.9 mm to (13.3, 6.38)
- moved C40 4.50 mm to (41.5, 88.5)
- moved R43 2.50 mm to (41.6, 85.0)
- moved U9 2.50 mm to (55.1, 94.5)
- moved C41 2.08 mm to (41.5, 92.5), turned to 0 degrees
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Connections:
- net GND: now also TP1.2
- net N$77: now also TP1.1; no longer P11.1

Commit message: Added scope test points per signal list, Made edits per latest email(Jan 19,2016 03:31pm. Created scope test point symbol footprint and component. Edited rowetel.lbr to make resistor & capacitor components consistent. Movinf power supply related components onto PCB to start layout. RGB
Parts:
- removed P12: TPAD50, _Coherix:TPAD50
- removed TP1: SCOPE_PAD, _RoweTel:SCOPE_PAD
- added SP1, SP2, SP3, SP4, SP5, SP6, SP7, SP8, SP9: SCOPE_PAD, _RoweTel:SCOPE_PAD
- C23, C26: value CAP-10UF-WJ5 -> .33uF,25V; device _RoweTel:NICHICON-WJ-5 -> _RoweTel:C0603
- C24, C25, C29, C37, C40, C41, C44, C45: device _RoweTel:C0805 -> _RoweTel:C0603
- C27, C28, C30, C33, C35, C39: device _RoweTel:C0805 -> _RoweTel:C0402
- C38: value 2.2uF,16V -> 2.2uF,25V; device _RoweTel:C0805 -> _RoweTel:C0402
- C42, C43: device _RoweTel:C1210 -> _RoweTel:C0603
- C46: device AA-ipc-7351-capacitor:CAPC1608X92N -> _RoweTel:C0603
- J2: value HDR100-5 -> HDR100-7; device _RoweTel:HDR100-5 -> _RoweTel:HDR100-7
- Q11: value BRF92 -> BFR92
- Q14, Q15: device transistor:SOT23-EBC -> _RoweTel:SOT23
- Q17: device transistor-pnp:TO5 -> _RoweTel:SOT23
- R1, R10, R11, R12, R13, R14, R16, R17, R18, R2, R21, R22, R24, R25, R26, R27, R28, R29, R3, R30, R34, R4, R40, R44, R46, R47, R5, R50, R54, R55, R56, R57, R6, R7, R8, R9: device _RoweTel:R0805 -> _RoweTel:R0402
- R19, R20, R23, R33, R35, R36, R38, R42, R43, R51, R52: device AA-ipc-7351-resistor:RESC1005X40AN -> _RoweTel:R0402
- R31, R32, R41, R45, R53: device AA-ipc-7351-resistor:RESC1608X55N -> _RoweTel:R0402
Connections:
- removed net AIN_PWR: C97.2, D10.1
- removed net N$110: Q17.3, R118.2
- removed net TX2NDLO: C121.2, C128.1
- new net AIN3: C97.2, D10.1, U1.26
- net +12VRXENB: now also J2.7
- net +12VTXENB: now also J2.6
- net 1ST_LO: now also SP6.1
- net AIN1: now also Q17.3, R118.2, SP1.1
- net AIN2: now also SP2.1; no longer P12.1
- net DAC2_OUT: now also SP4.1
- net GND: now also SP1.2, SP2.2, SP3.2, SP4.2, SP5.2, SP6.2, SP7.2, SP8.2, SP9.2; no longer TP1.2
- net N$105: now also Q17.1; no longer Q17.2
- net N$106: now also Q17.2; no longer Q17.1
- net N$140: now also Q15.3; no longer Q15.C
- net N$141: now also Q14.3, Q15.1; no longer Q14.C, Q15.B
- net N$146: now also Q14.1; no longer Q14.B
- net N$147: now also Q14.2; no longer Q14.E
- net N$148: now also Q15.2; no longer Q15.E
- net N$77: now also SP9.1; no longer TP1.1
- net RX-2ND-LO: now also C128.1, SP8.1
- net TX-2ND-LO: now also C121.2, SP7.1
- net TX_DAC: now also SP3.1, U1.29; no longer U1.32
- net VGG: now also SP5.1

Commit message: Progress - Latest PCB block layouts. Plocks are identified and are moveable. Present loations are placeholders. Added netlist(NET-SM2000.txt),PDF schematic(SCH_SM2000.pdf) BOM PDF(BOM-SM2000.txt) and PDF of board file(BRD-SM2000.pdf). RGB
Parts:
- removed P13: TPAD50, _Coherix:TPAD50
- added C137, C138: 100nF,25V, _RoweTel:C0805
- added FB20: FB0805, _RoweTel:FE0805
- C17, C18: value 2.2uF,16V -> 2.2uF,25V
- C22: value 4.7uF,16V,TANT -> 4.7uF,25V; device _RoweTel:C1206-TANT -> _RoweTel:C0805
- C23, C24, C25, C40, C45, C46: device _RoweTel:C0603 -> _RoweTel:C0805
- C26: value .33uF,25V -> 22uF,25V; device _RoweTel:C0603 -> _RoweTel:C1210
- C27: value 1nF,25V,0402 -> 1nF,25V; device _RoweTel:C0402 -> _RoweTel:C0805
- C28, C30, C33, C35, C38, C39: device _RoweTel:C0402 -> _RoweTel:C0805
- C29: value 100nF,25V -> 22uF,25V; device _RoweTel:C0603 -> _RoweTel:C1210
- C37, C41: value 1nF,25V -> 100nF,25V; device _RoweTel:C0603 -> _RoweTel:C0805
- C42, C43: device _RoweTel:C0603 -> _RoweTel:C1210
- C44: value 1uF,25V -> 22uF,25V; device _RoweTel:C0603 -> _RoweTel:C1210
- C47: device AA-ipc-7351-capacitor:CAPC1608X92N -> _RoweTel:C0805
- C48, C49, C51: device AA-ipc-7351-capacitor:CAPC1005X60N -> _RoweTel:C0805
- C50: value 3.9nF,16V -> 3.9nF,25V
- C6, C7: value 1uF,16V -> 1uF,25V
- C77: value 1uF,25V,EL -> 1uF,25V; device _RoweTel:C1206-TANT -> _RoweTel:C0805
- C95: value 22pF,25V -> 22pF,50V
- C99: value 1nF,25V -> 1nF,25V,DNL
- L18: value 9.2uH -> L-TDK-MLF-2012-9.2uH
- R1, R10, R11, R12, R13, R14, R16, R17, R18, R19, R2, R20, R21, R22, R23, R24, R25, R26, R27, R28, R29, R3, R30, R31, R32, R33, R34, R35, R36, R38, R4, R40, R41, R42, R43, R44, R45, R46, R5, R50, R51, R52, R53, R54, R55, R57, R6, R7, R8, R9: device _RoweTel:R0402 -> _RoweTel:R0805
- R37: device AA-ipc-7351-resistor:RESC1005X40AN -> _RoweTel:R0805
- R47, R56: value 2.2K,1/8W,5% -> 2.2K,1%; device _RoweTel:R0402 -> _RoweTel:R0805
- R49: device AA-ipc-7351-resistor:RESC3115X70N -> _RoweTel:R1206
- U5: value L78MXX -> L78M09
- U6: value L78MXX -> LD1117AS-33; device _RoweTel:DPAK -> _RoweTel:SOT223
- U8: value AP7215Y-33 -> LD1117AS-33; device _RoweTel:SOT89 -> _RoweTel:SOT223
- moved R21 275.4 mm to (147.3, 25.3)
- moved R74 268.4 mm to (151.0, 70.5), turned to 270 degrees
- moved R99 267.9 mm to (145.0, 53.5), turned to 180 degrees
- moved R76 267.2 mm to (146.0, 70.5), turned to 90 degrees
- moved R71 267.1 mm to (153.5, 70.5), turned to 270 degrees
- moved R98 266.1 mm to (145.0, 41.0), turned to 180 degrees
- moved R100 262.4 mm to (145.0, 51.0), turned to 180 degrees
- moved R75 260.1 mm to (151.0, 76.5), turned to 270 degrees
- moved R101 259.1 mm to (145.0, 56.0)
- moved C63 257.6 mm to (143.5, 70.5), turned to 90 degrees
- moved C58 256.4 mm to (136.0, 70.5), turned to 90 degrees
- moved U14 255.6 mm to (136.5, 49.5), turned to 270 degrees
- moved R96 251.5 mm to (145.0, 46.0), turned to 180 degrees
- moved C65 251.4 mm to (143.5, 63.5), turned to 270 degrees
- moved R73 250.1 mm to (148.5, 76.5), turned to 90 degrees
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Connections:
- removed net N$399: C40.1, C41.1, C42.1, C43.1, R41.2, R43.1, U9.2
- new net N$110: C137.1, C26.1, FB20.2, U6.3
- new net N$150: R41.1, SW5.2, SW5.3, SW5.5, SW5.6
- net +5V: now also FB20.1; no longer C26.1, U6.1
- net +VIN: now also C40.1, C41.1, C42.1, C43.1, R41.2, R43.1, U9.2; no longer R41.1, SW5.2, SW5.3, SW5.5, SW5.6
- net 1ST_LO: now also U11.1
- net 3V3: now also C37.1, U6.2, U6.4; no longer U6.3
- net A3V3: now also U8.2, U8.4; no longer U8.3
- net DAC2_OUT: no longer P13.1
- net GND: now also C137.2, C138.2, L18.P$2, U6.1; no longer L18.P$1, U6.4
- net N$145: now also L18.P$1; no longer L18.P$2
- net N$54: now also C138.1, U8.3; no longer C37.1, U8.2
Routing:
- net GND: track 0.00 -> 17.9 mm, vias 4 -> 19
- net N$129: track 0.00 -> 17.9 mm
- net N$77: track 0.00 -> 16.9 mm
- net +VIN: track 0.00 -> 6.28 mm, vias 0 -> 1
- net SW: track 0.00 -> 2.38 mm, vias 0 -> 8
- added copper zone on layer 1, net +5V
- added copper zone on layer 1, net +VIN
- added copper zone on layer 1, net GND
- added copper zone on layer 1, net SW
Other:
- board text added: "+9V"
- board text added: "3V3"
- board text added: "A3V3"
- board text added: "BASEBAND AMP"
- board text added: "LOCAL OSCILLATOR"
- board text added: "MIC PREAMP"
- board text added: "OTG USB INTERFACE"
- board text added: "RX+12V"
- board text added: "SPEAKER AMP"
- board text added: "TIA"
- board text added: "TX+12V"
- board text added: "XTAL 2ND MIXER"
