File: sm2000/SM2000-A/SM2000-A.brd (EAGLE design)
At the start: 160 x 160 mm, 452 parts, among them CN1 HDR100-3, CN2 ST-3509, CN3 HDR100-3, CN4 JS-MU3-002, CN5 DS-0518, CN6 ST-3509, CN7 ST-3509, J1 JMP-2PIN, J10 JMPR-2X2, J11 JMPR-2X2, J12 JMPR-2X2, J13 JMPR-2X2, J14 JMPR-2X2, J2 HDR100-7, J3 JMP-2PIN, J4 CONN-BOOM-XH-2A, J5 JMP-2PIN, J6 JMPR-2X2, J7 JMPR-2X2, J8 JMPR-2X2, J9 JMPR-2X2, P6 TPAD50, P7 TPAD50, P8 TPAD50, P9 TPAD50, Q1 MMBT3904, Q10 MMBT3904, Q11 BFR92, Q12 BFQ19, Q13 RD01MUS2, Q14 MMBT3904, Q15 MMBT3904, Q16 MMBT3904, Q17 MMBT3906, Q2 STR2P3LLH6, Q3 MMBT3904, Q4 STR2P3LLH6, Q5 MMBT3904, Q6 MMBT3904, Q7 MMBT3904, Q8 MMBT3904, Q9 MMBT3904, SW1 TS-02B, SW2 SW-LC2259, SW3 TS-026, SW4 TS-026, SW5 SW-LC2259EENP, U1 STM32F405VGT6, U10 LM386M-1, U11 ADE-1, U12 PGA-103+, U13 LMV341, U14 SI5351A, U15 SI570, U16 SA612A, U2 STMPS2141, U3 EMIF02-USB03F2, U4 DNL, U5 L78M09, U6 LD1117AS-33, U7 LMV341, U8 LD1117AS-33, U9 TPS54329E, X1 BU-SMA-H

Commit message: RELEASE TO PRODUCTION SM2000-A FILES
Parts:
- removed S13, S19, S32, S33, S34, S41, S42, S7: SGND, _RoweTel:SGND
- added C139, C140, C141, C142, C143: TBD, _RoweTel:C0805
- added C144: 100nF,25V, _RoweTel:C0805
- added DRILEGEND: (no value), drilegend:DRILEGEND
- added R123, R124, R125, R126, R127: TBD, _RoweTel:R0805
- C116, C88: value 8nF,50V -> 8.2nF,25V
- C13: value 1nF,25V -> TBD
- moved SP5 102.1 mm to (134.0, 108.0), turned to 180 degrees
- moved XTAL2 64.5 mm to (98.0, 74.0)
- moved C113 59.6 mm to (96.5, 68.5)
- moved C114 54.8 mm to (91.5, 74.5), turned to 180 degrees
- moved FB19 51.7 mm to (146.0, 119.5), turned to 180 degrees
- moved U14 46.0 mm to (91.5, 69.0), turned to 180 degrees
- moved R120 45.8 mm to (144.0, 115.5), turned to 180 degrees
- moved C136 45.5 mm to (150.0, 115.0), turned to 90 degrees
- moved C13 43.1 mm to (146.0, 122.5)
- moved R100 42.4 mm to (96.5, 61.5)
- moved R102 42.0 mm to (100.5, 61.5)
- moved R101 41.2 mm to (100.5, 65.0)
- moved R99 41.2 mm to (96.5, 65.0)
- moved C134 40.9 mm to (144.0, 112.0), turned to 0 degrees
- moved FB14 40.5 mm to (71.5, 75.5)
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Connections:
- removed net TIA_OUT: C70.1, C71.2, J9.1
- new net N$12: J6.2, U11.2
- new net N$139: C142.1, FB11.1, R127.1
- new net N$65: C70.1, C71.2, J9.2
- new net XAIN3: R123.1, U1.26
- new net XSCL3: R124.1, R29.2, U1.67, U4.6
- new net XSDA3: R125.1, R28.2, U1.66, U4.5
- new net XTX_DAC: R126.1, U1.29
- net 1ST_LO: now also U11.6; no longer U11.1
- net AIN3: now also C143.1, R123.2; no longer U1.26
- net BBAMP: now also C144.1; no longer C135.2, L20.P$2
- net GND: now also C139.2, C140.2, C141.2, C142.2, C143.2, C83.R1, C83.R2, U11.1, U11.4, U11.5; no longer C83.S, J6.3, S13.1, S19.1, S32.1, S33.1, S34.1, S41.1, S42.1, S7.1
- net N$145: now also C83.S; no longer C83.R1, C83.R2
- net N$90: now also C135.2, C144.2, L20.P$2; no longer J6.2, U11.5
- net SCL3: now also C139.1, R124.2; no longer R29.2, U1.67, U4.6
- net SDA3: now also C140.1, R125.2; no longer R28.2, U1.66, U4.5
- net TIAOUT: now also J9.1; no longer J9.2
- net TX_DAC: now also C141.1, R126.2; no longer U1.29
- net VGG: now also R127.2; no longer FB11.1
Routing:
- net VGG: track 187.8 -> 21.8 mm, vias 2 -> 1
- net N$139: track 0.00 -> 126.6 mm, vias 0 -> 2
- net RX+12V: track 7.95 -> 112.3 mm, vias 1 -> 2
- net TX+12V: track 99.3 -> 199.3 mm
- net AIN3: track 4.38 -> 96.7 mm, vias 0 -> 2
- net +5V: track 319.6 -> 256.9 mm
- net TX_DAC: track 98.4 -> 38.2 mm
- net RX-2ND-LO: track 89.9 -> 38.2 mm, vias 1 -> 2
- net XSCL3: track 0.00 -> 51.6 mm, vias 0 -> 2
- net GND: track 478.2 -> 521.1 mm, vias 140 -> 148
- net TIA_OUT: track 42.3 -> 0.00 mm
- net TX-2ND-LO: track 66.1 -> 25.2 mm, vias 0 -> 1
- net XSDA3: track 0.00 -> 40.5 mm, vias 0 -> 4
- net XAIN3: track 0.00 -> 39.0 mm, vias 0 -> 2
- net 1ST_LO: track 17.5 -> 51.8 mm
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- removed copper zone on layer 15, net SW
Other:
- board text added: "01-16"
- board text added: "01-20"
- board text added: "Copyright c 2016"
- board text added: "KA8BMA VK5KA VK5DGR"
- board text added: "L1-SM2000-A-503-A"
- board text added: "L2-SM2000-A-503-A"
- board text added: "L3-SM2000-A-503-A"
- board text added: "L4-SM2000-A-503-A"
- board text added: "LAYER-STACK"
- board text added: "Licensed under TAPR Open Hardware License"
- board text added: "Richard Barnich, Neil Abraham and David Rowe"
- board text added: "SM2000 - Digital Voice Tranceiver"
- board text added: "SM2000 Rev A"
- board text removed: "L1-SM2000-A-419"
- board text removed: "L2-SM2000-A-419"
- board text removed: "L3-SM2000-A-419"
- board text removed: "L4-SM2000-A-419"
