File: sm2000/SM2000-A/SM2000-A.sch (EAGLE design)
At the start: 452 parts, among them CN1 HDR100-3, CN2 ST-3509, CN3 HDR100-3, CN4 JS-MU3-002, CN5 DS-0518, CN6 ST-3509, CN7 ST-3509, J1 JMP-2PIN, J10 JMPR-2X2, J11 JMPR-2X2, J12 JMPR-2X2, J13 JMPR-2X2, J14 JMPR-2X2, J2 HDR100-7, J3 JMP-2PIN, J4 CONN-BOOM-XH-2A, J5 JMP-2PIN, J6 JMPR-2X2, J7 JMPR-2X2, J8 JMPR-2X2, J9 JMPR-2X2, P6 TPAD50, P7 TPAD50, P8 TPAD50, P9 TPAD50, Q1 MMBT3904, Q10 MMBT3904, Q11 BFR92, Q12 BFQ19, Q13 RD01MUS2, Q14 MMBT3904, Q15 MMBT3904, Q16 MMBT3904, Q17 MMBT3906, Q2 STR2P3LLH6, Q3 MMBT3904, Q4 STR2P3LLH6, Q5 MMBT3904, Q6 MMBT3904, Q7 MMBT3904, Q8 MMBT3904, Q9 MMBT3904, SW1 TS-02B, SW2 SW-LC2259, SW3 TS-026, SW4 TS-026, SW5 SW-LC2259EENP, U1 STM32F405VGT6, U10 LM386M-1, U11 ADE-1, U12 PGA-103+, U13 LMV341, U14 SI5351A, U15 SI570, U16 SA612A, U2 STMPS2141, U3 EMIF02-USB03F2, U4 DNL, U5 L78M09, U6 LD1117AS-33, U7 LMV341, U8 LD1117AS-33, U9 TPS54329E, X1 BU-SMA-H

Commit message: RELEASE TO PRODUCTION SM2000-A FILES
Parts:
- removed S13, S19, S32, S33, S34, S41, S42, S7: SGND, _RoweTel:SGND
- added C139, C140, C141, C142, C143: TBD, _RoweTel:CAP-0805
- added C144: 100nF,25V, _RoweTel:CAP-0805
- added R123, R124, R125, R126, R127: TBD, _RoweTel:RES-0805
- C116, C88: value 8nF,50V -> 8.2nF,25V
- C13: value 1nF,25V -> TBD
Connections:
- removed net TIA_OUT: C70.1, C71.2, J9.1
- new net N$12: J6.2, U11.IF
- new net N$139: C142.1, FB11.1, R127.1
- new net N$65: C70.1, C71.2, J9.2
- new net XAIN3: R123.1, U1A.PA3
- new net XSCL3: R124.1, R29.2, U1A.PA8, U4.SCL
- new net XSDA3: R125.1, R28.2, U1A.PC9, U4.SDA
- new net XTX_DAC: R126.1, U1A.PA4
- net 1ST_LO: now also U11.LO; no longer U11.G1
- net AIN3: now also C143.1, R123.2; no longer U1A.PA3
- net BBAMP: now also C144.1; no longer C135.2, L20.2
- net GND: now also C139.2, C140.2, C141.2, C142.2, C143.2, C83.R, U11.G1, U11.G2, U11.G3; no longer C83.S, J6.3, S13.1, S19.1, S32.1, S33.1, S34.1, S41.1, S42.1, S7.1
- net N$145: now also C83.S; no longer C83.R
- net N$90: now also C135.2, C144.2, L20.2; no longer J6.2, U11.G3
- net SCL3: now also C139.1, R124.2; no longer R29.2, U1A.PA8, U4.SCL
- net SDA3: now also C140.1, R125.2; no longer R28.2, U1A.PC9, U4.SDA
- net TIAOUT: now also J9.1; no longer J9.2
- net TX_DAC: now also C141.1, R126.2; no longer U1A.PA4
- net VGG: now also R127.2; no longer FB11.1
Other:
- note added: "SM2000 Rev A"
- note removed: "Baseand AMP"
- moved on the sheet: C10, C116, C13, C88, J2, J6, P6, P7, P8, P9, R121, R122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
